File: hanover-7320-20-01.brd (EAGLE design)
At the start: 158 parts, among them IC1 74HC75D, IC11 4514D, IC14 4514D, IC17 4514D, IC2 4024D, IC20 4514D, IC23 4514D, IC26 4514D, IC3 74HC139D, IC4 4024D, IC5 4514D, IC8 4514D

Commit message: Populate diodes and coils
The coils are not the actual dots and are just placeholders until a library is created for the dots
Parts:
- added D100, D1000, D1001, D1002, D1003, D1004, D1005, D1006, D1007, D1008, D1009, D101, D1010, D1011, D1012, D1013, D1014, D1015, D1016, D1017, D1018, D1019, D102, D1020, D1021, D1022, D1023, D1024, D103, D104, D105, D106, D107, D108, D109, D110, D111, D112, D113, D114, D115, D116, D117, D118, D119, D120, D121, D122, D123, D124, D125, D126, D127, D128, D129, D130, D131, D132, D133, D134, D135, D136, D137, D138, D139, D140, D141, D142, D143, D144, D145, D146, D147, D148, D149, D150, D151, D152, D153, D154, D155, D156, D157, D158, D159, D160, D161, D162, D163, D164, D165, D166, D167, D168, D169, D170, D171, D172, D173, D174, D175, D176, D177, D178, D179, D180, D181, D182, D183, D184, D185, D186, D187, D188, D189, D190, D191, D192, D193, D194, D195, D196, D197, D198, D199, D200, D201, D202, D203, D204, D205, D206, D207, D208, D209, D210, D211, D212, D213, D214, D215, D216, D217, D218, D219, D220, D221, D222, D223, D224, D225, D226, D227, D228, D229, D230, D231, D232, D233, D234, D235, D236, D237, D238, D239, D240, D241, D242, D243, D244, D245, D246, D247, D248, D249, D250, D251, D252, D253, D254, D255, D256, D257, D258, D259, D260, D261, D262, D263, D264, D265, D266, D267, D268, D269, D270, D271, D272, D273, D274, D275, D276, D277, D278, D279, D280, D281, D282, D283, D284, D285, D286, D287, D288, D289, D290, D291, D292, D293, D294, D295, D296, D297, D298, D299, D300, D301, D302, D303, D304, D305, D306, D307, D308, D309, D310, D311, D312, D313, D314, D315, D316, D317, D318, D319, D320, D321, D322, D323, D324, D325, D326, D327, D328, D329, D330, D331, D332, D333, D334, D335, D336, D337, D338, D339, D340, D341, D342, D343, D344, D345, D346, D347, D348, D349, D350, D351, D352, D353, D354, D355, D356, D357, D358, D359, D360, D361, D362, D363, D364, D365, D366, D367, D368, D369, D370, D371, D372, D373, D374, D375, D376, D377, D378, D379, D380, D381, D382, D383, D384, D385, D386, D387, D388, D389, D390, D391, D392, D393, D394, D395, D396, D397, D398, D399, D400, D401, D402, D403, D404, D405, D406, D407, D408, D409, D410, D411, D412, D413, D414, D415, D416, D417, D418, D419, D420, D421, D422, D423, D424, D425, D426, D427, D428, D429, D430, D431, D432, D433, D434, D435, D436, D437, D438, D439, D440, D441, D442, D443, D444, D445, D446, D447, D448, D449, D450, D451, D452, D453, D454, D455, D456, D457, D458, D459, D460, D461, D462, D463, D464, D465, D466, D467, D468, D469, D470, D471, D472, D473, D474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: 200mA/70V, SparkFun-DiscreteSemi:SOT23-3
- added L100, L1000, L1001, L1002, L1003, L1004, L1005, L1006, L1007, L1008, L1009, L101, L1010, L1011, L1012, L1013, L1014, L1015, L1016, L1017, L1018, L1019, L102, L1020, L1021, L1022, L1023, L1024, L103, L104, L105, L106, L107, L108, L109, L110, L111, L112, L113, L114, L115, L116, L117, L118, L119, L120, L121, L122, L123, L124, L125, L126, L127, L128, L129, L130, L131, L132, L133, L134, L135, L136, L137, L138, L139, L140, L141, L142, L143, L144, L145, L146, L147, L148, L149, L150, L151, L152, L153, L154, L155, L156, L157, L158, L159, L160, L161, L162, L163, L164, L165, L166, L167, L168, L169, L170, L171, L172, L173, L174, L175, L176, L177, L178, L179, L180, L181, L182, L183, L184, L185, L186, L187, L188, L189, L190, L191, L192, L193, L194, L195, L196, L197, L198, L199, L200, L201, L202, L203, L204, L205, L206, L207, L208, L209, L210, L211, L212, L213, L214, L215, L216, L217, L218, L219, L220, L221, L222, L223, L224, L225, L226, L227, L228, L229, L230, L231, L232, L233, L234, L235, L236, L237, L238, L239, L240, L241, L242, L243, L244, L245, L246, L247, L248, L249, L250, L251, L252, L253, L254, L255, L256, L257, L258, L259, L260, L261, L262, L263, L264, L265, L266, L267, L268, L269, L270, L271, L272, L273, L274, L275, L276, L277, L278, L279, L280, L281, L282, L283, L284, L285, L286, L287, L288, L289, L290, L291, L292, L293, L294, L295, L296, L297, L298, L299, L300, L301, L302, L303, L304, L305, L306, L307, L308, L309, L310, L311, L312, L313, L314, L315, L316, L317, L318, L319, L320, L321, L322, L323, L324, L325, L326, L327, L328, L329, L330, L331, L332, L333, L334, L335, L336, L337, L338, L339, L340, L341, L342, L343, L344, L345, L346, L347, L348, L349, L350, L351, L352, L353, L354, L355, L356, L357, L358, L359, L360, L361, L362, L363, L364, L365, L366, L367, L368, L369, L370, L371, L372, L373, L374, L375, L376, L377, L378, L379, L380, L381, L382, L383, L384, L385, L386, L387, L388, L389, L390, L391, L392, L393, L394, L395, L396, L397, L398, L399, L400, L401, L402, L403, L404, L405, L406, L407, L408, L409, L410, L411, L412, L413, L414, L415, L416, L417, L418, L419, L420, L421, L422, L423, L424, L425, L426, L427, L428, L429, L430, L431, L432, L433, L434, L435, L436, L437, L438, L439, L440, L441, L442, L443, L444, L445, L446, L447, L448, L449, L450, L451, L452, L453, L454, L455, L456, L457, L458, L459, L460, L461, L462, L463, L464, L465, L466, L467, L468, L469, L470, L471, L472, L473, L474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: (no value), inductor-neosid:SD8
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Connections:
- new net N$100: D86.3, L86.1
- new net N$1000: D986.3, L986.1
- new net N$1001: D987.3, L987.1
- new net N$1002: D988.3, L988.1
- new net N$1003: D989.3, L989.1
- new net N$1004: D990.3, L990.1
- new net N$1005: D991.3, L991.1
- new net N$1006: D992.3, L992.1
- new net N$1007: D993.3, L993.1
- new net N$1008: D994.3, L994.1
- new net N$1009: D995.3, L995.1
- new net N$101: D87.3, L87.1
- new net N$1010: D996.3, L996.1
- new net N$1011: D997.3, L997.1
- new net N$1012: D998.3, L998.1
- new net N$1013: D999.3, L999.1
- new net N$1014: D1000.3, L1000.1
- new net N$1015: D1001.3, L1001.1
- new net N$1016: D1002.3, L1002.1
- new net N$1017: D1003.3, L1003.1
- new net N$1018: D1004.3, L1004.1
- new net N$1019: D1005.3, L1005.1
- new net N$102: D88.3, L88.1
- new net N$1020: D1006.3, L1006.1
- new net N$1021: D1007.3, L1007.1
- new net N$1022: D1008.3, L1008.1
- new net N$1023: D1009.3, L1009.1
- new net N$1024: D1010.3, L1010.1
- new net N$1025: D1011.3, L1011.1
- new net N$1026: D1012.3, L1012.1
- new net N$1027: D1013.3, L1013.1
- new net N$1028: D1014.3, L1014.1
- new net N$1029: D1015.3, L1015.1
- new net N$103: D89.3, L89.1
- new net N$1030: D1016.3, L1016.1
- new net N$1031: D1017.3, L1017.1
- new net N$1032: D1018.3, L1018.1
- new net N$1033: D1019.3, L1019.1
- new net N$1034: D1020.3, L1020.1
- new net N$1035: D1021.3, L1021.1
- new net N$1036: D1022.3, L1022.1
- new net N$1037: D1023.3, L1023.1
- new net N$1038: D1024.3, L1024.1
- new net N$104: D90.3, L90.1
- new net N$105: D91.3, L91.1
- new net N$106: D92.3, L92.1
- new net N$107: D93.3, L93.1
- new net N$108: D94.3, L94.1
- new net N$109: D95.3, L95.1
- new net N$110: D96.3, L96.1
- new net N$111: D97.3, L97.1
- new net N$112: D98.3, L98.1
- new net N$113: D99.3, L99.1
- new net N$114: D100.3, L100.1
- new net N$115: D101.3, L101.1
- new net N$116: D102.3, L102.1
- new net N$117: D103.3, L103.1
- new net N$118: D104.3, L104.1
- new net N$119: D105.3, L105.1
- new net N$120: D106.3, L106.1
- new net N$121: D107.3, L107.1
- new net N$122: D108.3, L108.1
- new net N$123: D109.3, L109.1
- new net N$124: D110.3, L110.1
- new net N$125: D111.3, L111.1
- new net N$126: D112.3, L112.1
- new net N$127: D113.3, L113.1
- new net N$128: D114.3, L114.1
- new net N$129: D115.3, L115.1
- new net N$130: D116.3, L116.1
- new net N$131: D117.3, L117.1
- new net N$132: D118.3, L118.1
- new net N$133: D119.3, L119.1
- new net N$134: D120.3, L120.1
- new net N$135: D121.3, L121.1
- new net N$136: D122.3, L122.1
- new net N$137: D123.3, L123.1
- new net N$138: D124.3, L124.1
- new net N$139: D125.3, L125.1
- new net N$140: D126.3, L126.1
- new net N$141: D127.3, L127.1
- new net N$142: D128.3, L128.1
- new net N$143: D129.3, L129.1
- new net N$144: D130.3, L130.1
- new net N$145: D131.3, L131.1
- new net N$146: D132.3, L132.1
- new net N$147: D133.3, L133.1
- new net N$148: D134.3, L134.1
- new net N$149: D135.3, L135.1
- new net N$150: D136.3, L136.1
- new net N$151: D137.3, L137.1
- new net N$152: D138.3, L138.1
- new net N$153: D139.3, L139.1
- new net N$154: D140.3, L140.1
- new net N$155: D141.3, L141.1
- new net N$156: D142.3, L142.1
- new net N$157: D143.3, L143.1
- new net N$158: D144.3, L144.1
- new net N$159: D145.3, L145.1
- new net N$160: D146.3, L146.1
- new net N$161: D147.3, L147.1
- new net N$162: D148.3, L148.1
- new net N$163: D149.3, L149.1
- new net N$164: D150.3, L150.1
- new net N$165: D151.3, L151.1
- new net N$166: D152.3, L152.1
- new net N$167: D153.3, L153.1
- new net N$168: D154.3, L154.1
- new net N$169: D155.3, L155.1
- new net N$170: D156.3, L156.1
- new net N$171: D157.3, L157.1
- new net N$172: D158.3, L158.1
- new net N$173: D159.3, L159.1
- new net N$174: D160.3, L160.1
- new net N$175: D161.3, L161.1
- new net N$176: D162.3, L162.1
- new net N$177: D163.3, L163.1
- new net N$178: D164.3, L164.1
- new net N$179: D165.3, L165.1
- new net N$180: D166.3, L166.1
- new net N$181: D167.3, L167.1
- new net N$182: D168.3, L168.1
- new net N$183: D169.3, L169.1
- new net N$184: D170.3, L170.1
- new net N$185: D171.3, L171.1
- new net N$186: D172.3, L172.1
- new net N$187: D173.3, L173.1
- new net N$188: D174.3, L174.1
- new net N$189: D175.3, L175.1
- new net N$190: D176.3, L176.1
- new net N$191: D177.3, L177.1
- new net N$192: D178.3, L178.1
- new net N$193: D179.3, L179.1
- new net N$194: D180.3, L180.1
- new net N$195: D181.3, L181.1
- new net N$196: D182.3, L182.1
- new net N$197: D183.3, L183.1
- new net N$198: D184.3, L184.1
- new net N$199: D185.3, L185.1
- new net N$200: D186.3, L186.1
- new net N$201: D187.3, L187.1
- new net N$202: D188.3, L188.1
- new net N$203: D189.3, L189.1
- new net N$204: D190.3, L190.1
- new net N$205: D191.3, L191.1
- new net N$206: D192.3, L192.1
- new net N$207: D193.3, L193.1
- new net N$208: D194.3, L194.1
- new net N$209: D195.3, L195.1
- new net N$210: D196.3, L196.1
- new net N$211: D197.3, L197.1
- new net N$212: D198.3, L198.1
- new net N$213: D199.3, L199.1
- new net N$214: D200.3, L200.1
- new net N$215: D201.3, L201.1
- new net N$216: D202.3, L202.1
- new net N$217: D203.3, L203.1
- new net N$218: D204.3, L204.1
- new net N$219: D205.3, L205.1
- new net N$220: D206.3, L206.1
- new net N$221: D207.3, L207.1
- new net N$222: D208.3, L208.1
- new net N$223: D209.3, L209.1
- new net N$224: D210.3, L210.1
- new net N$225: D211.3, L211.1
- new net N$226: D212.3, L212.1
- new net N$227: D213.3, L213.1
- new net N$228: D214.3, L214.1
- new net N$229: D215.3, L215.1
- new net N$230: D216.3, L216.1
- new net N$231: D217.3, L217.1
- new net N$232: D218.3, L218.1
- new net N$233: D219.3, L219.1
- new net N$234: D220.3, L220.1
- new net N$235: D221.3, L221.1
- new net N$236: D222.3, L222.1
- new net N$237: D223.3, L223.1
- new net N$238: D224.3, L224.1
- new net N$239: D225.3, L225.1
- new net N$240: D226.3, L226.1
- new net N$241: D227.3, L227.1
- new net N$242: D228.3, L228.1
- new net N$243: D229.3, L229.1
- new net N$244: D230.3, L230.1
- new net N$245: D231.3, L231.1
- new net N$246: D232.3, L232.1
- new net N$247: D233.3, L233.1
- new net N$248: D234.3, L234.1
- new net N$249: D235.3, L235.1
- new net N$250: D236.3, L236.1
- new net N$251: D237.3, L237.1
- new net N$252: D238.3, L238.1
- new net N$253: D239.3, L239.1
- new net N$254: D240.3, L240.1
- new net N$255: D241.3, L241.1
- new net N$256: D242.3, L242.1
- new net N$257: D243.3, L243.1
- new net N$258: D244.3, L244.1
- new net N$259: D245.3, L245.1
- new net N$260: D246.3, L246.1
- new net N$261: D247.3, L247.1
- new net N$262: D248.3, L248.1
- new net N$263: D249.3, L249.1
- new net N$264: D250.3, L250.1
- new net N$265: D251.3, L251.1
- new net N$266: D252.3, L252.1
- new net N$267: D253.3, L253.1
- new net N$268: D254.3, L254.1
- new net N$269: D255.3, L255.1
- new net N$270: D256.3, L256.1
- new net N$271: D257.3, L257.1
- new net N$272: D258.3, L258.1
- new net N$273: D259.3, L259.1
- new net N$274: D260.3, L260.1
- new net N$275: D261.3, L261.1
- new net N$276: D262.3, L262.1
- new net N$277: D263.3, L263.1
- new net N$278: D264.3, L264.1
- new net N$279: D265.3, L265.1
- new net N$280: D266.3, L266.1
- new net N$281: D267.3, L267.1
- new net N$282: D268.3, L268.1
- new net N$283: D269.3, L269.1
- new net N$284: D270.3, L270.1
- new net N$285: D271.3, L271.1
- new net N$286: D272.3, L272.1
- new net N$287: D273.3, L273.1
- new net N$288: D274.3, L274.1
- new net N$289: D275.3, L275.1
- new net N$290: D276.3, L276.1
- new net N$291: D277.3, L277.1
- new net N$292: D278.3, L278.1
- new net N$293: D279.3, L279.1
- new net N$294: D280.3, L280.1
- new net N$295: D281.3, L281.1
- new net N$296: D282.3, L282.1
- new net N$297: D283.3, L283.1
- new net N$298: D284.3, L284.1
- new net N$299: D285.3, L285.1
- new net N$300: D286.3, L286.1
- new net N$301: D287.3, L287.1
- new net N$302: D288.3, L288.1
- new net N$303: D289.3, L289.1
- new net N$304: D290.3, L290.1
- new net N$305: D291.3, L291.1
- new net N$306: D292.3, L292.1
- new net N$307: D293.3, L293.1
- new net N$308: D294.3, L294.1
- new net N$309: D295.3, L295.1
- new net N$310: D296.3, L296.1
- new net N$311: D297.3, L297.1
- new net N$312: D298.3, L298.1
- new net N$313: D299.3, L299.1
- new net N$314: D300.3, L300.1
- new net N$315: D301.3, L301.1
- new net N$316: D302.3, L302.1
- new net N$317: D303.3, L303.1
- new net N$318: D304.3, L304.1
- new net N$319: D305.3, L305.1
- new net N$320: D306.3, L306.1
- new net N$321: D307.3, L307.1
- new net N$322: D308.3, L308.1
- new net N$323: D309.3, L309.1
- new net N$324: D310.3, L310.1
- new net N$325: D311.3, L311.1
- new net N$326: D312.3, L312.1
- new net N$327: D313.3, L313.1
- new net N$328: D314.3, L314.1
- new net N$329: D315.3, L315.1
- new net N$330: D316.3, L316.1
- new net N$331: D317.3, L317.1
- new net N$332: D318.3, L318.1
- new net N$333: D319.3, L319.1
- new net N$334: D320.3, L320.1
- new net N$335: D321.3, L321.1
- new net N$336: D322.3, L322.1
- new net N$337: D323.3, L323.1
- new net N$338: D324.3, L324.1
- new net N$339: D325.3, L325.1
- new net N$340: D326.3, L326.1
- new net N$341: D327.3, L327.1
- new net N$342: D328.3, L328.1
- new net N$343: D329.3, L329.1
- new net N$344: D330.3, L330.1
- new net N$345: D331.3, L331.1
- new net N$346: D332.3, L332.1
- new net N$347: D333.3, L333.1
- new net N$348: D334.3, L334.1
- new net N$349: D335.3, L335.1
- new net N$350: D336.3, L336.1
- new net N$351: D337.3, L337.1
- new net N$352: D338.3, L338.1
- new net N$353: D339.3, L339.1
- new net N$354: D340.3, L340.1
- new net N$355: D341.3, L341.1
- new net N$356: D342.3, L342.1
- new net N$357: D343.3, L343.1
- new net N$358: D344.3, L344.1
- new net N$359: D345.3, L345.1
- new net N$360: D346.3, L346.1
- new net N$361: D347.3, L347.1
- new net N$362: D348.3, L348.1
- new net N$363: D349.3, L349.1
- new net N$364: D350.3, L350.1
- new net N$365: D351.3, L351.1
- new net N$366: D352.3, L352.1
- new net N$367: D353.3, L353.1
- new net N$368: D354.3, L354.1
- new net N$369: D355.3, L355.1
- new net N$370: D356.3, L356.1
- new net N$371: D357.3, L357.1
- new net N$372: D358.3, L358.1
- new net N$373: D359.3, L359.1
- new net N$374: D360.3, L360.1
- new net N$375: D361.3, L361.1
- new net N$376: D362.3, L362.1
- new net N$377: D363.3, L363.1
- new net N$378: D364.3, L364.1
- new net N$379: D365.3, L365.1
- new net N$380: D366.3, L366.1
- new net N$381: D367.3, L367.1
- new net N$382: D368.3, L368.1
- new net N$383: D369.3, L369.1
- new net N$384: D370.3, L370.1
- new net N$385: D371.3, L371.1
- new net N$386: D372.3, L372.1
- new net N$387: D373.3, L373.1
- new net N$388: D374.3, L374.1
- new net N$389: D375.3, L375.1
- new net N$390: D376.3, L376.1
- new net N$391: D377.3, L377.1
- new net N$392: D378.3, L378.1
- new net N$393: D379.3, L379.1
- new net N$394: D380.3, L380.1
- new net N$395: D381.3, L381.1
- new net N$396: D382.3, L382.1
- new net N$397: D383.3, L383.1
- new net N$398: D384.3, L384.1
- new net N$399: D385.3, L385.1
- new net N$400: D386.3, L386.1
- new net N$401: D387.3, L387.1
- new net N$402: D388.3, L388.1
- new net N$403: D389.3, L389.1
- new net N$404: D390.3, L390.1
- new net N$405: D391.3, L391.1
- new net N$406: D392.3, L392.1
- new net N$407: D393.3, L393.1
- new net N$408: D394.3, L394.1
- new net N$409: D395.3, L395.1
- new net N$410: D396.3, L396.1
- new net N$411: D397.3, L397.1
- new net N$412: D398.3, L398.1
- new net N$413: D399.3, L399.1
- new net N$414: D400.3, L400.1
- new net N$415: D401.3, L401.1
- new net N$416: D402.3, L402.1
- new net N$417: D403.3, L403.1
- new net N$418: D404.3, L404.1
- new net N$419: D405.3, L405.1
- new net N$420: D406.3, L406.1
- new net N$421: D407.3, L407.1
- new net N$422: D408.3, L408.1
- new net N$423: D409.3, L409.1
- new net N$424: D410.3, L410.1
- new net N$425: D411.3, L411.1
- new net N$426: D412.3, L412.1
- new net N$427: D413.3, L413.1
- new net N$428: D414.3, L414.1
- new net N$429: D415.3, L415.1
- new net N$430: D416.3, L416.1
- new net N$431: D417.3, L417.1
- new net N$432: D418.3, L418.1
- new net N$433: D419.3, L419.1
- new net N$434: D420.3, L420.1
- new net N$435: D421.3, L421.1
- new net N$436: D422.3, L422.1
- new net N$437: D423.3, L423.1
- new net N$438: D424.3, L424.1
- new net N$439: D425.3, L425.1
- new net N$440: D426.3, L426.1
- new net N$441: D427.3, L427.1
- new net N$442: D428.3, L428.1
- new net N$443: D429.3, L429.1
- new net N$444: D430.3, L430.1
- new net N$445: D431.3, L431.1
- new net N$446: D432.3, L432.1
- new net N$447: D433.3, L433.1
- new net N$448: D434.3, L434.1
- new net N$449: D435.3, L435.1
- new net N$450: D436.3, L436.1
- new net N$451: D437.3, L437.1
- new net N$452: D438.3, L438.1
- new net N$453: D439.3, L439.1
- new net N$454: D440.3, L440.1
- new net N$455: D441.3, L441.1
- new net N$456: D442.3, L442.1
- new net N$457: D443.3, L443.1
- new net N$458: D444.3, L444.1
- new net N$459: D445.3, L445.1
- new net N$460: D446.3, L446.1
- new net N$461: D447.3, L447.1
- new net N$462: D448.3, L448.1
- new net N$463: D449.3, L449.1
- new net N$464: D450.3, L450.1
- new net N$465: D451.3, L451.1
- new net N$466: D452.3, L452.1
- new net N$467: D453.3, L453.1
- new net N$468: D454.3, L454.1
- new net N$469: D455.3, L455.1
- new net N$470: D456.3, L456.1
- new net N$471: D457.3, L457.1
- new net N$472: D458.3, L458.1
- new net N$473: D459.3, L459.1
- new net N$474: D460.3, L460.1
- new net N$475: D461.3, L461.1
- new net N$476: D462.3, L462.1
- new net N$477: D463.3, L463.1
- new net N$478: D464.3, L464.1
- new net N$479: D465.3, L465.1
- new net N$480: D466.3, L466.1
- new net N$481: D467.3, L467.1
- new net N$482: D468.3, L468.1
- new net N$483: D469.3, L469.1
- new net N$484: D470.3, L470.1
- new net N$485: D471.3, L471.1
- new net N$486: D472.3, L472.1
- new net N$487: D473.3, L473.1
- new net N$488: D474.3, L474.1
- new net N$489: D475.3, L475.1
- new net N$490: D476.3, L476.1
- new net N$491: D477.3, L477.1
- new net N$492: D478.3, L478.1
- new net N$493: D479.3, L479.1
- new net N$494: D480.3, L480.1
- new net N$495: D481.3, L481.1
- new net N$496: D482.3, L482.1
- new net N$497: D483.3, L483.1
- new net N$498: D484.3, L484.1
- new net N$499: D485.3, L485.1
- new net N$500: D486.3, L486.1
- new net N$501: D487.3, L487.1
- new net N$502: D488.3, L488.1
- new net N$503: D489.3, L489.1
- new net N$504: D490.3, L490.1
- new net N$505: D491.3, L491.1
- new net N$506: D492.3, L492.1
- new net N$507: D493.3, L493.1
- new net N$508: D494.3, L494.1
- new net N$509: D495.3, L495.1
- new net N$510: D496.3, L496.1
- new net N$511: D497.3, L497.1
- new net N$512: D498.3, L498.1
- new net N$513: D499.3, L499.1
- new net N$514: D500.3, L500.1
- new net N$515: D501.3, L501.1
- new net N$516: D502.3, L502.1
- new net N$517: D503.3, L503.1
- new net N$518: D504.3, L504.1
- new net N$519: D505.3, L505.1
- new net N$520: D506.3, L506.1
- new net N$521: D507.3, L507.1
- new net N$522: D508.3, L508.1
- new net N$523: D509.3, L509.1
- new net N$524: D510.3, L510.1
- new net N$525: D511.3, L511.1
- new net N$526: D512.3, L512.1
- new net N$527: D513.3, L513.1
- new net N$528: D514.3, L514.1
- new net N$529: D515.3, L515.1
- new net N$530: D516.3, L516.1
- new net N$531: D517.3, L517.1
- new net N$532: D518.3, L518.1
- new net N$533: D519.3, L519.1
- new net N$534: D520.3, L520.1
- new net N$535: D521.3, L521.1
- new net N$536: D522.3, L522.1
- new net N$537: D523.3, L523.1
- new net N$538: D524.3, L524.1
- new net N$539: D525.3, L525.1
- new net N$540: D526.3, L526.1
- new net N$541: D527.3, L527.1
- new net N$542: D528.3, L528.1
- new net N$543: D529.3, L529.1
- new net N$544: D530.3, L530.1
- new net N$545: D531.3, L531.1
- new net N$546: D532.3, L532.1
- new net N$547: D533.3, L533.1
- new net N$548: D534.3, L534.1
- new net N$549: D535.3, L535.1
- new net N$550: D536.3, L536.1
- new net N$551: D537.3, L537.1
- new net N$552: D538.3, L538.1
- new net N$553: D539.3, L539.1
- new net N$554: D540.3, L540.1
- new net N$555: D541.3, L541.1
- new net N$556: D542.3, L542.1
- new net N$557: D543.3, L543.1
- new net N$558: D544.3, L544.1
- new net N$559: D545.3, L545.1
- new net N$560: D546.3, L546.1
- new net N$561: D547.3, L547.1
- new net N$562: D548.3, L548.1
- new net N$563: D549.3, L549.1
- new net N$564: D550.3, L550.1
- new net N$565: D551.3, L551.1
- new net N$566: D552.3, L552.1
- new net N$567: D553.3, L553.1
- new net N$568: D554.3, L554.1
- new net N$569: D555.3, L555.1
- new net N$570: D556.3, L556.1
- new net N$571: D557.3, L557.1
- new net N$572: D558.3, L558.1
- new net N$573: D559.3, L559.1
- new net N$574: D560.3, L560.1
- new net N$575: D561.3, L561.1
- new net N$576: D562.3, L562.1
- new net N$577: D563.3, L563.1
- new net N$578: D564.3, L564.1
- new net N$579: D565.3, L565.1
- new net N$580: D566.3, L566.1
- new net N$581: D567.3, L567.1
- new net N$582: D568.3, L568.1
- new net N$583: D569.3, L569.1
- new net N$584: D570.3, L570.1
- new net N$585: D571.3, L571.1
- new net N$586: D572.3, L572.1
- new net N$587: D573.3, L573.1
- new net N$588: D574.3, L574.1
- new net N$589: D575.3, L575.1
- new net N$590: D576.3, L576.1
- new net N$591: D577.3, L577.1
- new net N$592: D578.3, L578.1
- new net N$593: D579.3, L579.1
- new net N$594: D580.3, L580.1
- new net N$595: D581.3, L581.1
- new net N$596: D582.3, L582.1
- new net N$597: D583.3, L583.1
- new net N$598: D584.3, L584.1
- new net N$599: D585.3, L585.1
- new net N$600: D586.3, L586.1
- new net N$601: D587.3, L587.1
- new net N$602: D588.3, L588.1
- new net N$603: D589.3, L589.1
- new net N$604: D590.3, L590.1
- new net N$605: D591.3, L591.1
- new net N$606: D592.3, L592.1
- new net N$607: D593.3, L593.1
- new net N$608: D594.3, L594.1
- new net N$609: D595.3, L595.1
- new net N$610: D596.3, L596.1
- new net N$611: D597.3, L597.1
- new net N$612: D598.3, L598.1
- new net N$613: D599.3, L599.1
- new net N$614: D600.3, L600.1
- new net N$615: D601.3, L601.1
- new net N$616: D602.3, L602.1
- new net N$617: D603.3, L603.1
- new net N$618: D604.3, L604.1
- new net N$619: D605.3, L605.1
- new net N$620: D606.3, L606.1
- new net N$621: D607.3, L607.1
- new net N$622: D608.3, L608.1
- new net N$623: D609.3, L609.1
- new net N$624: D610.3, L610.1
- new net N$625: D611.3, L611.1
- new net N$626: D612.3, L612.1
- new net N$627: D613.3, L613.1
- new net N$628: D614.3, L614.1
- new net N$629: D615.3, L615.1
- new net N$630: D616.3, L616.1
- new net N$631: D617.3, L617.1
- new net N$632: D618.3, L618.1
- new net N$633: D619.3, L619.1
- new net N$634: D620.3, L620.1
- new net N$635: D621.3, L621.1
- new net N$636: D622.3, L622.1
- new net N$637: D623.3, L623.1
- new net N$638: D624.3, L624.1
- new net N$639: D625.3, L625.1
- new net N$640: D626.3, L626.1
- new net N$641: D627.3, L627.1
- new net N$642: D628.3, L628.1
- new net N$643: D629.3, L629.1
- new net N$644: D630.3, L630.1
- new net N$645: D631.3, L631.1
- new net N$646: D632.3, L632.1
- new net N$647: D633.3, L633.1
- new net N$648: D634.3, L634.1
- new net N$649: D635.3, L635.1
- new net N$650: D636.3, L636.1
- new net N$651: D637.3, L637.1
- new net N$652: D638.3, L638.1
- new net N$653: D639.3, L639.1
- new net N$654: D640.3, L640.1
- new net N$655: D641.3, L641.1
- new net N$656: D642.3, L642.1
- new net N$657: D643.3, L643.1
- new net N$658: D644.3, L644.1
- new net N$659: D645.3, L645.1
- new net N$660: D646.3, L646.1
- new net N$661: D647.3, L647.1
- new net N$662: D648.3, L648.1
- new net N$663: D649.3, L649.1
- new net N$664: D650.3, L650.1
- new net N$665: D651.3, L651.1
- new net N$666: D652.3, L652.1
- new net N$667: D653.3, L653.1
- new net N$668: D654.3, L654.1
- new net N$669: D655.3, L655.1
- new net N$670: D656.3, L656.1
- new net N$671: D657.3, L657.1
- new net N$672: D658.3, L658.1
- new net N$673: D659.3, L659.1
- new net N$674: D660.3, L660.1
- new net N$675: D661.3, L661.1
- new net N$676: D662.3, L662.1
- new net N$677: D663.3, L663.1
- new net N$678: D664.3, L664.1
- new net N$679: D665.3, L665.1
- new net N$680: D666.3, L666.1
- new net N$681: D667.3, L667.1
- new net N$682: D668.3, L668.1
- new net N$683: D669.3, L669.1
- new net N$684: D670.3, L670.1
- new net N$685: D671.3, L671.1
- new net N$686: D672.3, L672.1
- new net N$687: D673.3, L673.1
- new net N$688: D674.3, L674.1
- new net N$689: D675.3, L675.1
- new net N$690: D676.3, L676.1
- new net N$691: D677.3, L677.1
- new net N$692: D678.3, L678.1
- new net N$693: D679.3, L679.1
- new net N$694: D680.3, L680.1
- new net N$695: D681.3, L681.1
- new net N$696: D682.3, L682.1
- new net N$697: D683.3, L683.1
- new net N$698: D684.3, L684.1
- new net N$699: D685.3, L685.1
- new net N$700: D686.3, L686.1
- new net N$701: D687.3, L687.1
- new net N$702: D688.3, L688.1
- new net N$703: D689.3, L689.1
- new net N$704: D690.3, L690.1
- new net N$705: D691.3, L691.1
- new net N$706: D692.3, L692.1
- new net N$707: D693.3, L693.1
- new net N$708: D694.3, L694.1
- new net N$709: D695.3, L695.1
- new net N$710: D696.3, L696.1
- new net N$711: D697.3, L697.1
- new net N$712: D698.3, L698.1
- new net N$713: D699.3, L699.1
- new net N$714: D700.3, L700.1
- new net N$715: D701.3, L701.1
- new net N$716: D702.3, L702.1
- new net N$717: D703.3, L703.1
- new net N$718: D704.3, L704.1
- new net N$719: D705.3, L705.1
- new net N$720: D706.3, L706.1
- new net N$721: D707.3, L707.1
- new net N$722: D708.3, L708.1
- new net N$723: D709.3, L709.1
- new net N$724: D710.3, L710.1
- new net N$725: D711.3, L711.1
- new net N$726: D712.3, L712.1
- new net N$727: D713.3, L713.1
- new net N$728: D714.3, L714.1
- new net N$729: D715.3, L715.1
- new net N$730: D716.3, L716.1
- new net N$731: D717.3, L717.1
- new net N$732: D718.3, L718.1
- new net N$733: D719.3, L719.1
- new net N$734: D720.3, L720.1
- new net N$735: D721.3, L721.1
- new net N$736: D722.3, L722.1
- new net N$737: D723.3, L723.1
- new net N$738: D724.3, L724.1
- new net N$739: D725.3, L725.1
- new net N$740: D726.3, L726.1
- new net N$741: D727.3, L727.1
- new net N$742: D728.3, L728.1
- new net N$743: D729.3, L729.1
- new net N$744: D730.3, L730.1
- new net N$745: D731.3, L731.1
- new net N$746: D732.3, L732.1
- new net N$747: D733.3, L733.1
- new net N$748: D734.3, L734.1
- new net N$749: D735.3, L735.1
- new net N$750: D736.3, L736.1
- new net N$751: D737.3, L737.1
- new net N$752: D738.3, L738.1
- new net N$753: D739.3, L739.1
- new net N$754: D740.3, L740.1
- new net N$755: D741.3, L741.1
- new net N$756: D742.3, L742.1
- new net N$757: D743.3, L743.1
- new net N$758: D744.3, L744.1
- new net N$759: D745.3, L745.1
- new net N$760: D746.3, L746.1
- new net N$761: D747.3, L747.1
- new net N$762: D748.3, L748.1
- new net N$763: D749.3, L749.1
- new net N$764: D750.3, L750.1
- new net N$765: D751.3, L751.1
- new net N$766: D752.3, L752.1
- new net N$767: D753.3, L753.1
- new net N$768: D754.3, L754.1
- new net N$769: D755.3, L755.1
- new net N$770: D756.3, L756.1
- new net N$771: D757.3, L757.1
- new net N$772: D758.3, L758.1
- new net N$773: D759.3, L759.1
- new net N$774: D760.3, L760.1
- new net N$775: D761.3, L761.1
- new net N$776: D762.3, L762.1
- new net N$777: D763.3, L763.1
- new net N$778: D764.3, L764.1
- new net N$779: D765.3, L765.1
- new net N$780: D766.3, L766.1
- new net N$781: D767.3, L767.1
- new net N$782: D768.3, L768.1
- new net N$783: D769.3, L769.1
- new net N$784: D770.3, L770.1
- new net N$785: D771.3, L771.1
- new net N$786: D772.3, L772.1
- new net N$787: D773.3, L773.1
- new net N$788: D774.3, L774.1
- new net N$789: D775.3, L775.1
- new net N$79: D65.3, L65.1
- new net N$790: D776.3, L776.1
- new net N$791: D777.3, L777.1
- new net N$792: D778.3, L778.1
- new net N$793: D779.3, L779.1
- new net N$794: D780.3, L780.1
- new net N$795: D781.3, L781.1
- new net N$796: D782.3, L782.1
- new net N$797: D783.3, L783.1
- new net N$798: D784.3, L784.1
- new net N$799: D785.3, L785.1
- new net N$80: D66.3, L66.1
- new net N$800: D786.3, L786.1
- new net N$801: D787.3, L787.1
- new net N$802: D788.3, L788.1
- new net N$803: D789.3, L789.1
- new net N$804: D790.3, L790.1
- new net N$805: D791.3, L791.1
- new net N$806: D792.3, L792.1
- new net N$807: D793.3, L793.1
- new net N$808: D794.3, L794.1
- new net N$809: D795.3, L795.1
- new net N$81: D67.3, L67.1
- new net N$810: D796.3, L796.1
- new net N$811: D797.3, L797.1
- new net N$812: D798.3, L798.1
- new net N$813: D799.3, L799.1
- new net N$814: D800.3, L800.1
- new net N$815: D801.3, L801.1
- new net N$816: D802.3, L802.1
- new net N$817: D803.3, L803.1
- new net N$818: D804.3, L804.1
- new net N$819: D805.3, L805.1
- new net N$82: D68.3, L68.1
- new net N$820: D806.3, L806.1
- new net N$821: D807.3, L807.1
- new net N$822: D808.3, L808.1
- new net N$823: D809.3, L809.1
- new net N$824: D810.3, L810.1
- new net N$825: D811.3, L811.1
- new net N$826: D812.3, L812.1
- new net N$827: D813.3, L813.1
- new net N$828: D814.3, L814.1
- new net N$829: D815.3, L815.1
- new net N$83: D69.3, L69.1
- new net N$830: D816.3, L816.1
- new net N$831: D817.3, L817.1
- new net N$832: D818.3, L818.1
- new net N$833: D819.3, L819.1
- new net N$834: D820.3, L820.1
- new net N$835: D821.3, L821.1
- new net N$836: D822.3, L822.1
- new net N$837: D823.3, L823.1
- new net N$838: D824.3, L824.1
- new net N$839: D825.3, L825.1
- new net N$84: D70.3, L70.1
- new net N$840: D826.3, L826.1
- new net N$841: D827.3, L827.1
- new net N$842: D828.3, L828.1
- new net N$843: D829.3, L829.1
- new net N$844: D830.3, L830.1
- new net N$845: D831.3, L831.1
- new net N$846: D832.3, L832.1
- new net N$847: D833.3, L833.1
- new net N$848: D834.3, L834.1
- new net N$849: D835.3, L835.1
- new net N$85: D71.3, L71.1
- new net N$850: D836.3, L836.1
- new net N$851: D837.3, L837.1
- new net N$852: D838.3, L838.1
- new net N$853: D839.3, L839.1
- new net N$854: D840.3, L840.1
- new net N$855: D841.3, L841.1
- new net N$856: D842.3, L842.1
- new net N$857: D843.3, L843.1
- new net N$858: D844.3, L844.1
- new net N$859: D845.3, L845.1
- new net N$86: D72.3, L72.1
- new net N$860: D846.3, L846.1
- new net N$861: D847.3, L847.1
- new net N$862: D848.3, L848.1
- new net N$863: D849.3, L849.1
- new net N$864: D850.3, L850.1
- new net N$865: D851.3, L851.1
- new net N$866: D852.3, L852.1
- new net N$867: D853.3, L853.1
- new net N$868: D854.3, L854.1
- new net N$869: D855.3, L855.1
- new net N$87: D73.3, L73.1
- new net N$870: D856.3, L856.1
- new net N$871: D857.3, L857.1
- new net N$872: D858.3, L858.1
- new net N$873: D859.3, L859.1
- new net N$874: D860.3, L860.1
- new net N$875: D861.3, L861.1
- new net N$876: D862.3, L862.1
- new net N$877: D863.3, L863.1
- new net N$878: D864.3, L864.1
- new net N$879: D865.3, L865.1
- new net N$88: D74.3, L74.1
- new net N$880: D866.3, L866.1
- new net N$881: D867.3, L867.1
- new net N$882: D868.3, L868.1
- new net N$883: D869.3, L869.1
- new net N$884: D870.3, L870.1
- new net N$885: D871.3, L871.1
- new net N$886: D872.3, L872.1
- new net N$887: D873.3, L873.1
- new net N$888: D874.3, L874.1
- new net N$889: D875.3, L875.1
- new net N$89: D75.3, L75.1
- new net N$890: D876.3, L876.1
- new net N$891: D877.3, L877.1
- new net N$892: D878.3, L878.1
- new net N$893: D879.3, L879.1
- new net N$894: D880.3, L880.1
- new net N$895: D881.3, L881.1
- new net N$896: D882.3, L882.1
- new net N$897: D883.3, L883.1
- new net N$898: D884.3, L884.1
- new net N$899: D885.3, L885.1
- new net N$90: D76.3, L76.1
- new net N$900: D886.3, L886.1
- new net N$901: D887.3, L887.1
- new net N$902: D888.3, L888.1
- new net N$903: D889.3, L889.1
- new net N$904: D890.3, L890.1
- new net N$905: D891.3, L891.1
- new net N$906: D892.3, L892.1
- new net N$907: D893.3, L893.1
- new net N$908: D894.3, L894.1
- new net N$909: D895.3, L895.1
- new net N$91: D77.3, L77.1
- new net N$910: D896.3, L896.1
- new net N$911: D897.3, L897.1
- new net N$912: D898.3, L898.1
- new net N$913: D899.3, L899.1
- new net N$914: D900.3, L900.1
- new net N$915: D901.3, L901.1
- new net N$916: D902.3, L902.1
- new net N$917: D903.3, L903.1
- new net N$918: D904.3, L904.1
- new net N$919: D905.3, L905.1
- new net N$92: D78.3, L78.1
- new net N$920: D906.3, L906.1
- new net N$921: D907.3, L907.1
- new net N$922: D908.3, L908.1
- new net N$923: D909.3, L909.1
- new net N$924: D910.3, L910.1
- new net N$925: D911.3, L911.1
- new net N$926: D912.3, L912.1
- new net N$927: D913.3, L913.1
- new net N$928: D914.3, L914.1
- new net N$929: D915.3, L915.1
- new net N$93: D79.3, L79.1
- new net N$930: D916.3, L916.1
- new net N$931: D917.3, L917.1
- new net N$932: D918.3, L918.1
- new net N$933: D919.3, L919.1
- new net N$934: D920.3, L920.1
- new net N$935: D921.3, L921.1
- new net N$936: D922.3, L922.1
- new net N$937: D923.3, L923.1
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Other:
- board outline added: 160 x 100 mm

Commit message: Wired transistor arrays to correct 18V lines, separated diodes/coils schematic into 4 sheets, add frames
Connections:
- removed net 5V1: IC28.10
- removed net 5V2: IC16.10, IC19.10, IC22.10
- removed net 5V3: IC25.10
- removed net C13_SOURCE: IC17.14
- removed net C16_SOURCE: IC17.15
- removed net C17_SINK: IC20.11
- removed net C17_SOURCE: IC20.18
- removed net C18_SINK: IC20.9
- removed net C18_SOURCE: IC20.17
- removed net C19_SINK: IC20.10
- removed net C19_SOURCE: IC20.20
- removed net C1_SINK: IC14.11
- removed net C1_SOURCE: IC14.18
- removed net C20_SINK: IC20.8
- removed net C20_SOURCE: IC20.19
- removed net C21_SINK: IC20.7
- removed net C21_SOURCE: IC20.14
- removed net C22_SINK: IC20.6
- removed net C22_SOURCE: IC20.13
- removed net C23_SINK: IC20.5
- removed net C23_SOURCE: IC20.16
- removed net C24_SINK: IC20.4
- removed net C24_SOURCE: IC20.15
- removed net C25_SINK: IC23.11
- removed net C25_SOURCE: IC23.18
- removed net C26_SINK: IC23.9
- removed net C26_SOURCE: IC23.17
- removed net C27_SINK: IC23.10
- removed net C27_SOURCE: IC23.20
- removed net C28_SINK: IC23.8
- removed net C28_SOURCE: IC23.19
- removed net C29_SINK: IC23.7
- removed net C29_SOURCE: IC23.14
- removed net C2_SINK: IC14.9
- removed net C2_SOURCE: IC14.17
- removed net C30_SINK: IC23.6
- removed net C30_SOURCE: IC23.13
- removed net C31_SINK: IC23.5
- removed net C31_SOURCE: IC23.16
- removed net C32_SINK: IC23.4
- removed net C32_SOURCE: IC23.15
- removed net C3_SINK: IC14.10
- removed net C3_SOURCE: IC14.20
- removed net C4_SINK: IC14.8
- removed net C4_SOURCE: IC14.19
- removed net C5_SINK: IC14.7
- removed net C5_SOURCE: IC14.14
- removed net C6_SINK: IC14.6
- removed net C6_SOURCE: IC14.13
- removed net C7_SINK: IC14.5
- removed net C7_SOURCE: IC14.16
- removed net C8_SINK: IC14.4
- removed net C8_SOURCE: IC14.15
- removed net COL25_SINK: IC24.18
- removed net COL25_SOURCE: IC25.18
- removed net COL26_SINK: IC24.17
- removed net COL26_SOURCE: IC25.17
- removed net COL27_SINK: IC24.16
- removed net COL27_SOURCE: IC25.16
- removed net COL28_SINK: IC24.15
- removed net COL28_SOURCE: IC25.15
- removed net COL29_SINK: IC24.14
- removed net COL29_SOURCE: IC25.14
- removed net COL30_SINK: IC24.13
- removed net COL30_SOURCE: IC25.13
- removed net COL31_SINK: IC24.12
- removed net COL31_SOURCE: IC25.12
- removed net COL32_SINK: IC24.11
- removed net COL32_SOURCE: IC25.11
- removed net N$16: IC24.5
- removed net N$4: IC27.5
- removed net R1_SINK3: IC28.1
- removed net R1_SINK5: IC19.1
- removed net R1_SINK7: IC25.1
- removed net R1_SOURCE3: IC27.1
- removed net R1_SOURCE5: IC18.1
- removed net R1_SOURCE7: IC24.1
- removed net R2_SINK3: IC28.2
- removed net R2_SINK5: IC19.2
- removed net R2_SINK7: IC25.2
- removed net R2_SOURCE3: IC27.2
- removed net R2_SOURCE5: IC18.2
- removed net R2_SOURCE7: IC24.2
- removed net R3_SINK3: IC28.3
- removed net R3_SINK5: IC19.3
- removed net R3_SINK7: IC25.3
- removed net R3_SOURCE3: IC27.3
- removed net R3_SOURCE5: IC18.3
- removed net R3_SOURCE7: IC24.3
- removed net R4_SINK3: IC28.4
- removed net R4_SINK5: IC19.4
- removed net R4_SINK7: IC25.4
- removed net R4_SOURCE3: IC27.4
- removed net R4_SOURCE5: IC18.4
- removed net R4_SOURCE7: IC24.4
- removed net R5_SINK3: IC28.5
- removed net R5_SINK5: IC19.5
- removed net R5_SINK7: IC25.5
- removed net R6_SINK3: IC28.6
- removed net R6_SINK5: IC19.6
- removed net R6_SINK7: IC25.6
- removed net R6_SOURCE3: IC27.6
- removed net R6_SOURCE5: IC18.6
- removed net R6_SOURCE7: IC24.6
- removed net R7_SINK3: IC28.7
- removed net R7_SINK5: IC19.7
- removed net R7_SINK7: IC25.7
- removed net R7_SOURCE3: IC27.7
- removed net R7_SOURCE5: IC18.7
- removed net R7_SOURCE7: IC24.7
- removed net R8_SINK3: IC28.8
- removed net R8_SINK5: IC19.8
- removed net R8_SINK7: IC25.8
- removed net R8_SOURCE3: IC27.8
- removed net R8_SOURCE7: IC24.8
- removed net VCC: IC10.9, IC12.9, IC15.9, IC18.9, IC21.9, IC24.9, IC27.9, IC7.9
- new net R25_SINK1: IC23.11, IC25.1
- new net R25_SOURCE1: IC23.18, IC24.1
- new net R26_SINK1: IC23.9, IC25.2
- new net R26_SOURCE1: IC23.17, IC24.2
- new net R27_SINK1: IC23.10, IC25.3
- new net R27_SOURCE1: IC23.20, IC24.3
- new net R28_SINK1: IC23.8, IC25.4
- new net R28_SOURCE1: IC23.19, IC24.4
- new net R29_SINK1: IC23.7, IC25.5
- new net R29_SOURCE1: IC23.14, IC24.5
- new net R30_SINK1: IC23.6, IC25.6
- new net R30_SOURCE1: IC23.13, IC24.6
- new net R31_SINK1: IC23.5, IC25.7
- new net R31_SOURCE1: IC23.16, IC24.7
- new net R32_SINK1: IC23.4, IC25.8
- new net R32_SOURCE1: IC23.15, IC24.8
- net 18V_PULSE_1: now also IC10.9, IC12.9, IC13.10, IC15.9, IC18.9, IC21.9, IC24.9, IC27.9, IC28.10, IC6.10, IC7.9, IC9.10
- net 18V_PULSE_2: now also IC16.10, IC19.10, IC22.10, IC25.10
- net 5V: no longer IC13.10, IC6.10, IC9.10
- net C10_SINK: now also IC19.2
- net C10_SOURCE: now also IC18.2
- net C11_SINK: now also IC19.3
- net C11_SOURCE: now also IC18.3
- net C12_SINK: now also IC19.4
- net C12_SOURCE: now also IC18.4
- net C13_SINK: now also IC19.5
- net C14_SINK: now also IC19.6
- net C14_SOURCE: now also IC18.6
- net C15_SINK: now also IC19.7
- net C15_SOURCE: now also IC18.7
- net C16_SINK: now also IC19.8
- net C9_SINK: now also IC19.1
- net C9_SOURCE: now also IC18.1
- net COL25: now also IC24.18, IC25.18
- net COL26: now also IC24.17, IC25.17
- net COL27: now also IC24.16, IC25.16
- net COL28: now also IC24.15, IC25.15
- net COL29: now also IC24.14, IC25.14
- net COL30: now also IC24.13, IC25.13
- net COL31: now also IC24.12, IC25.12
- net COL32: now also IC24.11, IC25.11
- net N$11: now also IC14.14
- net N$13: now also IC17.14
- net N$14: now also IC20.14
- net R1_SINK4: now also IC14.11
- net R1_SINK6: now also IC20.11
- net R1_SOURCE4: now also IC14.18
- net R1_SOURCE6: now also IC20.18
- net R25_SINK: now also IC28.1
- net R25_SOURCE: now also IC27.1
- net R26_SINK: now also IC28.2
- net R26_SOURCE: now also IC27.2
- net R27_SINK: now also IC28.3
- net R27_SOURCE: now also IC27.3
- net R28_SINK: now also IC28.4
- net R28_SOURCE: now also IC27.4
- net R29_SINK: now also IC28.5
- net R29_SOURCE: now also IC27.5
- net R2_SINK4: now also IC14.9
- net R2_SINK6: now also IC20.9
- net R2_SOURCE4: now also IC14.17
- net R2_SOURCE6: now also IC20.17
- net R30_SINK: now also IC28.6
- net R30_SOURCE: now also IC27.6
- net R31_SINK: now also IC28.7
- net R31_SOURCE: now also IC27.7
- net R32_SINK: now also IC28.8
- net R32_SOURCE: now also IC27.8
- net R3_SINK4: now also IC14.10
- net R3_SINK6: now also IC20.10
- net R3_SOURCE4: now also IC14.20
- net R3_SOURCE6: now also IC20.20
- net R4_SINK4: now also IC14.8
- net R4_SINK6: now also IC20.8
- net R4_SOURCE4: now also IC14.19
- net R4_SOURCE6: now also IC20.19
- net R5_SINK4: now also IC14.7
- net R5_SINK6: now also IC20.7
- net R6_SINK4: now also IC14.6
- net R6_SINK6: now also IC20.6
- net R6_SOURCE4: now also IC14.13
- net R6_SOURCE6: now also IC20.13
- net R7_SINK4: now also IC14.5
- net R7_SINK6: now also IC20.5
- net R7_SOURCE4: now also IC14.16
- net R7_SOURCE6: now also IC20.16
- net R8_SINK4: now also IC14.4
- net R8_SINK6: now also IC20.4
- net R8_SOURCE4: now also IC14.15
- net R8_SOURCE5: now also IC17.15
- net R8_SOURCE6: now also IC20.15
