File: hanover-7320-20-01.sch (EAGLE design)
At the start: 158 parts, among them IC1 74HC75D, IC11 4514D, IC14 4514D, IC17 4514D, IC2 4024D, IC20 4514D, IC23 4514D, IC26 4514D, IC3 74HC139D, IC4 4024D, IC5 4514D, IC8 4514D

Commit message: Populate diodes and coils
The coils are not the actual dots and are just placeholders until a library is created for the dots
Parts:
- added D100, D1000, D1001, D1002, D1003, D1004, D1005, D1006, D1007, D1008, D1009, D101, D1010, D1011, D1012, D1013, D1014, D1015, D1016, D1017, D1018, D1019, D102, D1020, D1021, D1022, D1023, D1024, D103, D104, D105, D106, D107, D108, D109, D110, D111, D112, D113, D114, D115, D116, D117, D118, D119, D120, D121, D122, D123, D124, D125, D126, D127, D128, D129, D130, D131, D132, D133, D134, D135, D136, D137, D138, D139, D140, D141, D142, D143, D144, D145, D146, D147, D148, D149, D150, D151, D152, D153, D154, D155, D156, D157, D158, D159, D160, D161, D162, D163, D164, D165, D166, D167, D168, D169, D170, D171, D172, D173, D174, D175, D176, D177, D178, D179, D180, D181, D182, D183, D184, D185, D186, D187, D188, D189, D190, D191, D192, D193, D194, D195, D196, D197, D198, D199, D200, D201, D202, D203, D204, D205, D206, D207, D208, D209, D210, D211, D212, D213, D214, D215, D216, D217, D218, D219, D220, D221, D222, D223, D224, D225, D226, D227, D228, D229, D230, D231, D232, D233, D234, D235, D236, D237, D238, D239, D240, D241, D242, D243, D244, D245, D246, D247, D248, D249, D250, D251, D252, D253, D254, D255, D256, D257, D258, D259, D260, D261, D262, D263, D264, D265, D266, D267, D268, D269, D270, D271, D272, D273, D274, D275, D276, D277, D278, D279, D280, D281, D282, D283, D284, D285, D286, D287, D288, D289, D290, D291, D292, D293, D294, D295, D296, D297, D298, D299, D300, D301, D302, D303, D304, D305, D306, D307, D308, D309, D310, D311, D312, D313, D314, D315, D316, D317, D318, D319, D320, D321, D322, D323, D324, D325, D326, D327, D328, D329, D330, D331, D332, D333, D334, D335, D336, D337, D338, D339, D340, D341, D342, D343, D344, D345, D346, D347, D348, D349, D350, D351, D352, D353, D354, D355, D356, D357, D358, D359, D360, D361, D362, D363, D364, D365, D366, D367, D368, D369, D370, D371, D372, D373, D374, D375, D376, D377, D378, D379, D380, D381, D382, D383, D384, D385, D386, D387, D388, D389, D390, D391, D392, D393, D394, D395, D396, D397, D398, D399, D400, D401, D402, D403, D404, D405, D406, D407, D408, D409, D410, D411, D412, D413, D414, D415, D416, D417, D418, D419, D420, D421, D422, D423, D424, D425, D426, D427, D428, D429, D430, D431, D432, D433, D434, D435, D436, D437, D438, D439, D440, D441, D442, D443, D444, D445, D446, D447, D448, D449, D450, D451, D452, D453, D454, D455, D456, D457, D458, D459, D460, D461, D462, D463, D464, D465, D466, D467, D468, D469, D470, D471, D472, D473, D474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: 200mA/70V, SparkFun-DiscreteSemi:BAV99
- added L100, L1000, L1001, L1002, L1003, L1004, L1005, L1006, L1007, L1008, L1009, L101, L1010, L1011, L1012, L1013, L1014, L1015, L1016, L1017, L1018, L1019, L102, L1020, L1021, L1022, L1023, L1024, L103, L104, L105, L106, L107, L108, L109, L110, L111, L112, L113, L114, L115, L116, L117, L118, L119, L120, L121, L122, L123, L124, L125, L126, L127, L128, L129, L130, L131, L132, L133, L134, L135, L136, L137, L138, L139, L140, L141, L142, L143, L144, L145, L146, L147, L148, L149, L150, L151, L152, L153, L154, L155, L156, L157, L158, L159, L160, L161, L162, L163, L164, L165, L166, L167, L168, L169, L170, L171, L172, L173, L174, L175, L176, L177, L178, L179, L180, L181, L182, L183, L184, L185, L186, L187, L188, L189, L190, L191, L192, L193, L194, L195, L196, L197, L198, L199, L200, L201, L202, L203, L204, L205, L206, L207, L208, L209, L210, L211, L212, L213, L214, L215, L216, L217, L218, L219, L220, L221, L222, L223, L224, L225, L226, L227, L228, L229, L230, L231, L232, L233, L234, L235, L236, L237, L238, L239, L240, L241, L242, L243, L244, L245, L246, L247, L248, L249, L250, L251, L252, L253, L254, L255, L256, L257, L258, L259, L260, L261, L262, L263, L264, L265, L266, L267, L268, L269, L270, L271, L272, L273, L274, L275, L276, L277, L278, L279, L280, L281, L282, L283, L284, L285, L286, L287, L288, L289, L290, L291, L292, L293, L294, L295, L296, L297, L298, L299, L300, L301, L302, L303, L304, L305, L306, L307, L308, L309, L310, L311, L312, L313, L314, L315, L316, L317, L318, L319, L320, L321, L322, L323, L324, L325, L326, L327, L328, L329, L330, L331, L332, L333, L334, L335, L336, L337, L338, L339, L340, L341, L342, L343, L344, L345, L346, L347, L348, L349, L350, L351, L352, L353, L354, L355, L356, L357, L358, L359, L360, L361, L362, L363, L364, L365, L366, L367, L368, L369, L370, L371, L372, L373, L374, L375, L376, L377, L378, L379, L380, L381, L382, L383, L384, L385, L386, L387, L388, L389, L390, L391, L392, L393, L394, L395, L396, L397, L398, L399, L400, L401, L402, L403, L404, L405, L406, L407, L408, L409, L410, L411, L412, L413, L414, L415, L416, L417, L418, L419, L420, L421, L422, L423, L424, L425, L426, L427, L428, L429, L430, L431, L432, L433, L434, L435, L436, L437, L438, L439, L440, L441, L442, L443, L444, L445, L446, L447, L448, L449, L450, L451, L452, L453, L454, L455, L456, L457, L458, L459, L460, L461, L462, L463, L464, L465, L466, L467, L468, L469, L470, L471, L472, L473, L474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: (no value), inductor-neosid:SD8
Connections:
- new net N$100: D86.COM, L86.1
- new net N$1000: D986.COM, L986.1
- new net N$1001: D987.COM, L987.1
- new net N$1002: D988.COM, L988.1
- new net N$1003: D989.COM, L989.1
- new net N$1004: D990.COM, L990.1
- new net N$1005: D991.COM, L991.1
- new net N$1006: D992.COM, L992.1
- new net N$1007: D993.COM, L993.1
- new net N$1008: D994.COM, L994.1
- new net N$1009: D995.COM, L995.1
- new net N$101: D87.COM, L87.1
- new net N$1010: D996.COM, L996.1
- new net N$1011: D997.COM, L997.1
- new net N$1012: D998.COM, L998.1
- new net N$1013: D999.COM, L999.1
- new net N$1014: D1000.COM, L1000.1
- new net N$1015: D1001.COM, L1001.1
- new net N$1016: D1002.COM, L1002.1
- new net N$1017: D1003.COM, L1003.1
- new net N$1018: D1004.COM, L1004.1
- new net N$1019: D1005.COM, L1005.1
- new net N$102: D88.COM, L88.1
- new net N$1020: D1006.COM, L1006.1
- new net N$1021: D1007.COM, L1007.1
- new net N$1022: D1008.COM, L1008.1
- new net N$1023: D1009.COM, L1009.1
- new net N$1024: D1010.COM, L1010.1
- new net N$1025: D1011.COM, L1011.1
- new net N$1026: D1012.COM, L1012.1
- new net N$1027: D1013.COM, L1013.1
- new net N$1028: D1014.COM, L1014.1
- new net N$1029: D1015.COM, L1015.1
- new net N$103: D89.COM, L89.1
- new net N$1030: D1016.COM, L1016.1
- new net N$1031: D1017.COM, L1017.1
- new net N$1032: D1018.COM, L1018.1
- new net N$1033: D1019.COM, L1019.1
- new net N$1034: D1020.COM, L1020.1
- new net N$1035: D1021.COM, L1021.1
- new net N$1036: D1022.COM, L1022.1
- new net N$1037: D1023.COM, L1023.1
- new net N$1038: D1024.COM, L1024.1
- new net N$104: D90.COM, L90.1
- new net N$105: D91.COM, L91.1
- new net N$106: D92.COM, L92.1
- new net N$107: D93.COM, L93.1
- new net N$108: D94.COM, L94.1
- new net N$109: D95.COM, L95.1
- new net N$110: D96.COM, L96.1
- new net N$111: D97.COM, L97.1
- new net N$112: D98.COM, L98.1
- new net N$113: D99.COM, L99.1
- new net N$114: D100.COM, L100.1
- new net N$115: D101.COM, L101.1
- new net N$116: D102.COM, L102.1
- new net N$117: D103.COM, L103.1
- new net N$118: D104.COM, L104.1
- new net N$119: D105.COM, L105.1
- new net N$120: D106.COM, L106.1
- new net N$121: D107.COM, L107.1
- new net N$122: D108.COM, L108.1
- new net N$123: D109.COM, L109.1
- new net N$124: D110.COM, L110.1
- new net N$125: D111.COM, L111.1
- new net N$126: D112.COM, L112.1
- new net N$127: D113.COM, L113.1
- new net N$128: D114.COM, L114.1
- new net N$129: D115.COM, L115.1
- new net N$130: D116.COM, L116.1
- new net N$131: D117.COM, L117.1
- new net N$132: D118.COM, L118.1
- new net N$133: D119.COM, L119.1
- new net N$134: D120.COM, L120.1
- new net N$135: D121.COM, L121.1
- new net N$136: D122.COM, L122.1
- new net N$137: D123.COM, L123.1
- new net N$138: D124.COM, L124.1
- new net N$139: D125.COM, L125.1
- new net N$140: D126.COM, L126.1
- new net N$141: D127.COM, L127.1
- new net N$142: D128.COM, L128.1
- new net N$143: D129.COM, L129.1
- new net N$144: D130.COM, L130.1
- new net N$145: D131.COM, L131.1
- new net N$146: D132.COM, L132.1
- new net N$147: D133.COM, L133.1
- new net N$148: D134.COM, L134.1
- new net N$149: D135.COM, L135.1
- new net N$150: D136.COM, L136.1
- new net N$151: D137.COM, L137.1
- new net N$152: D138.COM, L138.1
- new net N$153: D139.COM, L139.1
- new net N$154: D140.COM, L140.1
- new net N$155: D141.COM, L141.1
- new net N$156: D142.COM, L142.1
- new net N$157: D143.COM, L143.1
- new net N$158: D144.COM, L144.1
- new net N$159: D145.COM, L145.1
- new net N$160: D146.COM, L146.1
- new net N$161: D147.COM, L147.1
- new net N$162: D148.COM, L148.1
- new net N$163: D149.COM, L149.1
- new net N$164: D150.COM, L150.1
- new net N$165: D151.COM, L151.1
- new net N$166: D152.COM, L152.1
- new net N$167: D153.COM, L153.1
- new net N$168: D154.COM, L154.1
- new net N$169: D155.COM, L155.1
- new net N$170: D156.COM, L156.1
- new net N$171: D157.COM, L157.1
- new net N$172: D158.COM, L158.1
- new net N$173: D159.COM, L159.1
- new net N$174: D160.COM, L160.1
- new net N$175: D161.COM, L161.1
- new net N$176: D162.COM, L162.1
- new net N$177: D163.COM, L163.1
- new net N$178: D164.COM, L164.1
- new net N$179: D165.COM, L165.1
- new net N$180: D166.COM, L166.1
- new net N$181: D167.COM, L167.1
- new net N$182: D168.COM, L168.1
- new net N$183: D169.COM, L169.1
- new net N$184: D170.COM, L170.1
- new net N$185: D171.COM, L171.1
- new net N$186: D172.COM, L172.1
- new net N$187: D173.COM, L173.1
- new net N$188: D174.COM, L174.1
- new net N$189: D175.COM, L175.1
- new net N$190: D176.COM, L176.1
- new net N$191: D177.COM, L177.1
- new net N$192: D178.COM, L178.1
- new net N$193: D179.COM, L179.1
- new net N$194: D180.COM, L180.1
- new net N$195: D181.COM, L181.1
- new net N$196: D182.COM, L182.1
- new net N$197: D183.COM, L183.1
- new net N$198: D184.COM, L184.1
- new net N$199: D185.COM, L185.1
- new net N$200: D186.COM, L186.1
- new net N$201: D187.COM, L187.1
- new net N$202: D188.COM, L188.1
- new net N$203: D189.COM, L189.1
- new net N$204: D190.COM, L190.1
- new net N$205: D191.COM, L191.1
- new net N$206: D192.COM, L192.1
- new net N$207: D193.COM, L193.1
- new net N$208: D194.COM, L194.1
- new net N$209: D195.COM, L195.1
- new net N$210: D196.COM, L196.1
- new net N$211: D197.COM, L197.1
- new net N$212: D198.COM, L198.1
- new net N$213: D199.COM, L199.1
- new net N$214: D200.COM, L200.1
- new net N$215: D201.COM, L201.1
- new net N$216: D202.COM, L202.1
- new net N$217: D203.COM, L203.1
- new net N$218: D204.COM, L204.1
- new net N$219: D205.COM, L205.1
- new net N$220: D206.COM, L206.1
- new net N$221: D207.COM, L207.1
- new net N$222: D208.COM, L208.1
- new net N$223: D209.COM, L209.1
- new net N$224: D210.COM, L210.1
- new net N$225: D211.COM, L211.1
- new net N$226: D212.COM, L212.1
- new net N$227: D213.COM, L213.1
- new net N$228: D214.COM, L214.1
- new net N$229: D215.COM, L215.1
- new net N$230: D216.COM, L216.1
- new net N$231: D217.COM, L217.1
- new net N$232: D218.COM, L218.1
- new net N$233: D219.COM, L219.1
- new net N$234: D220.COM, L220.1
- new net N$235: D221.COM, L221.1
- new net N$236: D222.COM, L222.1
- new net N$237: D223.COM, L223.1
- new net N$238: D224.COM, L224.1
- new net N$239: D225.COM, L225.1
- new net N$240: D226.COM, L226.1
- new net N$241: D227.COM, L227.1
- new net N$242: D228.COM, L228.1
- new net N$243: D229.COM, L229.1
- new net N$244: D230.COM, L230.1
- new net N$245: D231.COM, L231.1
- new net N$246: D232.COM, L232.1
- new net N$247: D233.COM, L233.1
- new net N$248: D234.COM, L234.1
- new net N$249: D235.COM, L235.1
- new net N$250: D236.COM, L236.1
- new net N$251: D237.COM, L237.1
- new net N$252: D238.COM, L238.1
- new net N$253: D239.COM, L239.1
- new net N$254: D240.COM, L240.1
- new net N$255: D241.COM, L241.1
- new net N$256: D242.COM, L242.1
- new net N$257: D243.COM, L243.1
- new net N$258: D244.COM, L244.1
- new net N$259: D245.COM, L245.1
- new net N$260: D246.COM, L246.1
- new net N$261: D247.COM, L247.1
- new net N$262: D248.COM, L248.1
- new net N$263: D249.COM, L249.1
- new net N$264: D250.COM, L250.1
- new net N$265: D251.COM, L251.1
- new net N$266: D252.COM, L252.1
- new net N$267: D253.COM, L253.1
- new net N$268: D254.COM, L254.1
- new net N$269: D255.COM, L255.1
- new net N$270: D256.COM, L256.1
- new net N$271: D257.COM, L257.1
- new net N$272: D258.COM, L258.1
- new net N$273: D259.COM, L259.1
- new net N$274: D260.COM, L260.1
- new net N$275: D261.COM, L261.1
- new net N$276: D262.COM, L262.1
- new net N$277: D263.COM, L263.1
- new net N$278: D264.COM, L264.1
- new net N$279: D265.COM, L265.1
- new net N$280: D266.COM, L266.1
- new net N$281: D267.COM, L267.1
- new net N$282: D268.COM, L268.1
- new net N$283: D269.COM, L269.1
- new net N$284: D270.COM, L270.1
- new net N$285: D271.COM, L271.1
- new net N$286: D272.COM, L272.1
- new net N$287: D273.COM, L273.1
- new net N$288: D274.COM, L274.1
- new net N$289: D275.COM, L275.1
- new net N$290: D276.COM, L276.1
- new net N$291: D277.COM, L277.1
- new net N$292: D278.COM, L278.1
- new net N$293: D279.COM, L279.1
- new net N$294: D280.COM, L280.1
- new net N$295: D281.COM, L281.1
- new net N$296: D282.COM, L282.1
- new net N$297: D283.COM, L283.1
- new net N$298: D284.COM, L284.1
- new net N$299: D285.COM, L285.1
- new net N$300: D286.COM, L286.1
- new net N$301: D287.COM, L287.1
- new net N$302: D288.COM, L288.1
- new net N$303: D289.COM, L289.1
- new net N$304: D290.COM, L290.1
- new net N$305: D291.COM, L291.1
- new net N$306: D292.COM, L292.1
- new net N$307: D293.COM, L293.1
- new net N$308: D294.COM, L294.1
- new net N$309: D295.COM, L295.1
- new net N$310: D296.COM, L296.1
- new net N$311: D297.COM, L297.1
- new net N$312: D298.COM, L298.1
- new net N$313: D299.COM, L299.1
- new net N$314: D300.COM, L300.1
- new net N$315: D301.COM, L301.1
- new net N$316: D302.COM, L302.1
- new net N$317: D303.COM, L303.1
- new net N$318: D304.COM, L304.1
- new net N$319: D305.COM, L305.1
- new net N$320: D306.COM, L306.1
- new net N$321: D307.COM, L307.1
- new net N$322: D308.COM, L308.1
- new net N$323: D309.COM, L309.1
- new net N$324: D310.COM, L310.1
- new net N$325: D311.COM, L311.1
- new net N$326: D312.COM, L312.1
- new net N$327: D313.COM, L313.1
- new net N$328: D314.COM, L314.1
- new net N$329: D315.COM, L315.1
- new net N$330: D316.COM, L316.1
- new net N$331: D317.COM, L317.1
- new net N$332: D318.COM, L318.1
- new net N$333: D319.COM, L319.1
- new net N$334: D320.COM, L320.1
- new net N$335: D321.COM, L321.1
- new net N$336: D322.COM, L322.1
- new net N$337: D323.COM, L323.1
- new net N$338: D324.COM, L324.1
- new net N$339: D325.COM, L325.1
- new net N$340: D326.COM, L326.1
- new net N$341: D327.COM, L327.1
- new net N$342: D328.COM, L328.1
- new net N$343: D329.COM, L329.1
- new net N$344: D330.COM, L330.1
- new net N$345: D331.COM, L331.1
- new net N$346: D332.COM, L332.1
- new net N$347: D333.COM, L333.1
- new net N$348: D334.COM, L334.1
- new net N$349: D335.COM, L335.1
- new net N$350: D336.COM, L336.1
- new net N$351: D337.COM, L337.1
- new net N$352: D338.COM, L338.1
- new net N$353: D339.COM, L339.1
- new net N$354: D340.COM, L340.1
- new net N$355: D341.COM, L341.1
- new net N$356: D342.COM, L342.1
- new net N$357: D343.COM, L343.1
- new net N$358: D344.COM, L344.1
- new net N$359: D345.COM, L345.1
- new net N$360: D346.COM, L346.1
- new net N$361: D347.COM, L347.1
- new net N$362: D348.COM, L348.1
- new net N$363: D349.COM, L349.1
- new net N$364: D350.COM, L350.1
- new net N$365: D351.COM, L351.1
- new net N$366: D352.COM, L352.1
- new net N$367: D353.COM, L353.1
- new net N$368: D354.COM, L354.1
- new net N$369: D355.COM, L355.1
- new net N$370: D356.COM, L356.1
- new net N$371: D357.COM, L357.1
- new net N$372: D358.COM, L358.1
- new net N$373: D359.COM, L359.1
- new net N$374: D360.COM, L360.1
- new net N$375: D361.COM, L361.1
- new net N$376: D362.COM, L362.1
- new net N$377: D363.COM, L363.1
- new net N$378: D364.COM, L364.1
- new net N$379: D365.COM, L365.1
- new net N$380: D366.COM, L366.1
- new net N$381: D367.COM, L367.1
- new net N$382: D368.COM, L368.1
- new net N$383: D369.COM, L369.1
- new net N$384: D370.COM, L370.1
- new net N$385: D371.COM, L371.1
- new net N$386: D372.COM, L372.1
- new net N$387: D373.COM, L373.1
- new net N$388: D374.COM, L374.1
- new net N$389: D375.COM, L375.1
- new net N$390: D376.COM, L376.1
- new net N$391: D377.COM, L377.1
- new net N$392: D378.COM, L378.1
- new net N$393: D379.COM, L379.1
- new net N$394: D380.COM, L380.1
- new net N$395: D381.COM, L381.1
- new net N$396: D382.COM, L382.1
- new net N$397: D383.COM, L383.1
- new net N$398: D384.COM, L384.1
- new net N$399: D385.COM, L385.1
- new net N$400: D386.COM, L386.1
- new net N$401: D387.COM, L387.1
- new net N$402: D388.COM, L388.1
- new net N$403: D389.COM, L389.1
- new net N$404: D390.COM, L390.1
- new net N$405: D391.COM, L391.1
- new net N$406: D392.COM, L392.1
- new net N$407: D393.COM, L393.1
- new net N$408: D394.COM, L394.1
- new net N$409: D395.COM, L395.1
- new net N$410: D396.COM, L396.1
- new net N$411: D397.COM, L397.1
- new net N$412: D398.COM, L398.1
- new net N$413: D399.COM, L399.1
- new net N$414: D400.COM, L400.1
- new net N$415: D401.COM, L401.1
- new net N$416: D402.COM, L402.1
- new net N$417: D403.COM, L403.1
- new net N$418: D404.COM, L404.1
- new net N$419: D405.COM, L405.1
- new net N$420: D406.COM, L406.1
- new net N$421: D407.COM, L407.1
- new net N$422: D408.COM, L408.1
- new net N$423: D409.COM, L409.1
- new net N$424: D410.COM, L410.1
- new net N$425: D411.COM, L411.1
- new net N$426: D412.COM, L412.1
- new net N$427: D413.COM, L413.1
- new net N$428: D414.COM, L414.1
- new net N$429: D415.COM, L415.1
- new net N$430: D416.COM, L416.1
- new net N$431: D417.COM, L417.1
- new net N$432: D418.COM, L418.1
- new net N$433: D419.COM, L419.1
- new net N$434: D420.COM, L420.1
- new net N$435: D421.COM, L421.1
- new net N$436: D422.COM, L422.1
- new net N$437: D423.COM, L423.1
- new net N$438: D424.COM, L424.1
- new net N$439: D425.COM, L425.1
- new net N$440: D426.COM, L426.1
- new net N$441: D427.COM, L427.1
- new net N$442: D428.COM, L428.1
- new net N$443: D429.COM, L429.1
- new net N$444: D430.COM, L430.1
- new net N$445: D431.COM, L431.1
- new net N$446: D432.COM, L432.1
- new net N$447: D433.COM, L433.1
- new net N$448: D434.COM, L434.1
- new net N$449: D435.COM, L435.1
- new net N$450: D436.COM, L436.1
- new net N$451: D437.COM, L437.1
- new net N$452: D438.COM, L438.1
- new net N$453: D439.COM, L439.1
- new net N$454: D440.COM, L440.1
- new net N$455: D441.COM, L441.1
- new net N$456: D442.COM, L442.1
- new net N$457: D443.COM, L443.1
- new net N$458: D444.COM, L444.1
- new net N$459: D445.COM, L445.1
- new net N$460: D446.COM, L446.1
- new net N$461: D447.COM, L447.1
- new net N$462: D448.COM, L448.1
- new net N$463: D449.COM, L449.1
- new net N$464: D450.COM, L450.1
- new net N$465: D451.COM, L451.1
- new net N$466: D452.COM, L452.1
- new net N$467: D453.COM, L453.1
- new net N$468: D454.COM, L454.1
- new net N$469: D455.COM, L455.1
- new net N$470: D456.COM, L456.1
- new net N$471: D457.COM, L457.1
- new net N$472: D458.COM, L458.1
- new net N$473: D459.COM, L459.1
- new net N$474: D460.COM, L460.1
- new net N$475: D461.COM, L461.1
- new net N$476: D462.COM, L462.1
- new net N$477: D463.COM, L463.1
- new net N$478: D464.COM, L464.1
- new net N$479: D465.COM, L465.1
- new net N$480: D466.COM, L466.1
- new net N$481: D467.COM, L467.1
- new net N$482: D468.COM, L468.1
- new net N$483: D469.COM, L469.1
- new net N$484: D470.COM, L470.1
- new net N$485: D471.COM, L471.1
- new net N$486: D472.COM, L472.1
- new net N$487: D473.COM, L473.1
- new net N$488: D474.COM, L474.1
- new net N$489: D475.COM, L475.1
- new net N$490: D476.COM, L476.1
- new net N$491: D477.COM, L477.1
- new net N$492: D478.COM, L478.1
- new net N$493: D479.COM, L479.1
- new net N$494: D480.COM, L480.1
- new net N$495: D481.COM, L481.1
- new net N$496: D482.COM, L482.1
- new net N$497: D483.COM, L483.1
- new net N$498: D484.COM, L484.1
- new net N$499: D485.COM, L485.1
- new net N$500: D486.COM, L486.1
- new net N$501: D487.COM, L487.1
- new net N$502: D488.COM, L488.1
- new net N$503: D489.COM, L489.1
- new net N$504: D490.COM, L490.1
- new net N$505: D491.COM, L491.1
- new net N$506: D492.COM, L492.1
- new net N$507: D493.COM, L493.1
- new net N$508: D494.COM, L494.1
- new net N$509: D495.COM, L495.1
- new net N$510: D496.COM, L496.1
- new net N$511: D497.COM, L497.1
- new net N$512: D498.COM, L498.1
- new net N$513: D499.COM, L499.1
- new net N$514: D500.COM, L500.1
- new net N$515: D501.COM, L501.1
- new net N$516: D502.COM, L502.1
- new net N$517: D503.COM, L503.1
- new net N$518: D504.COM, L504.1
- new net N$519: D505.COM, L505.1
- new net N$520: D506.COM, L506.1
- new net N$521: D507.COM, L507.1
- new net N$522: D508.COM, L508.1
- new net N$523: D509.COM, L509.1
- new net N$524: D510.COM, L510.1
- new net N$525: D511.COM, L511.1
- new net N$526: D512.COM, L512.1
- new net N$527: D513.COM, L513.1
- new net N$528: D514.COM, L514.1
- new net N$529: D515.COM, L515.1
- new net N$530: D516.COM, L516.1
- new net N$531: D517.COM, L517.1
- new net N$532: D518.COM, L518.1
- new net N$533: D519.COM, L519.1
- new net N$534: D520.COM, L520.1
- new net N$535: D521.COM, L521.1
- new net N$536: D522.COM, L522.1
- new net N$537: D523.COM, L523.1
- new net N$538: D524.COM, L524.1
- new net N$539: D525.COM, L525.1
- new net N$540: D526.COM, L526.1
- new net N$541: D527.COM, L527.1
- new net N$542: D528.COM, L528.1
- new net N$543: D529.COM, L529.1
- new net N$544: D530.COM, L530.1
- new net N$545: D531.COM, L531.1
- new net N$546: D532.COM, L532.1
- new net N$547: D533.COM, L533.1
- new net N$548: D534.COM, L534.1
- new net N$549: D535.COM, L535.1
- new net N$550: D536.COM, L536.1
- new net N$551: D537.COM, L537.1
- new net N$552: D538.COM, L538.1
- new net N$553: D539.COM, L539.1
- new net N$554: D540.COM, L540.1
- new net N$555: D541.COM, L541.1
- new net N$556: D542.COM, L542.1
- new net N$557: D543.COM, L543.1
- new net N$558: D544.COM, L544.1
- new net N$559: D545.COM, L545.1
- new net N$560: D546.COM, L546.1
- new net N$561: D547.COM, L547.1
- new net N$562: D548.COM, L548.1
- new net N$563: D549.COM, L549.1
- new net N$564: D550.COM, L550.1
- new net N$565: D551.COM, L551.1
- new net N$566: D552.COM, L552.1
- new net N$567: D553.COM, L553.1
- new net N$568: D554.COM, L554.1
- new net N$569: D555.COM, L555.1
- new net N$570: D556.COM, L556.1
- new net N$571: D557.COM, L557.1
- new net N$572: D558.COM, L558.1
- new net N$573: D559.COM, L559.1
- new net N$574: D560.COM, L560.1
- new net N$575: D561.COM, L561.1
- new net N$576: D562.COM, L562.1
- new net N$577: D563.COM, L563.1
- new net N$578: D564.COM, L564.1
- new net N$579: D565.COM, L565.1
- new net N$580: D566.COM, L566.1
- new net N$581: D567.COM, L567.1
- new net N$582: D568.COM, L568.1
- new net N$583: D569.COM, L569.1
- new net N$584: D570.COM, L570.1
- new net N$585: D571.COM, L571.1
- new net N$586: D572.COM, L572.1
- new net N$587: D573.COM, L573.1
- new net N$588: D574.COM, L574.1
- new net N$589: D575.COM, L575.1
- new net N$590: D576.COM, L576.1
- new net N$591: D577.COM, L577.1
- new net N$592: D578.COM, L578.1
- new net N$593: D579.COM, L579.1
- new net N$594: D580.COM, L580.1
- new net N$595: D581.COM, L581.1
- new net N$596: D582.COM, L582.1
- new net N$597: D583.COM, L583.1
- new net N$598: D584.COM, L584.1
- new net N$599: D585.COM, L585.1
- new net N$600: D586.COM, L586.1
- new net N$601: D587.COM, L587.1
- new net N$602: D588.COM, L588.1
- new net N$603: D589.COM, L589.1
- new net N$604: D590.COM, L590.1
- new net N$605: D591.COM, L591.1
- new net N$606: D592.COM, L592.1
- new net N$607: D593.COM, L593.1
- new net N$608: D594.COM, L594.1
- new net N$609: D595.COM, L595.1
- new net N$610: D596.COM, L596.1
- new net N$611: D597.COM, L597.1
- new net N$612: D598.COM, L598.1
- new net N$613: D599.COM, L599.1
- new net N$614: D600.COM, L600.1
- new net N$615: D601.COM, L601.1
- new net N$616: D602.COM, L602.1
- new net N$617: D603.COM, L603.1
- new net N$618: D604.COM, L604.1
- new net N$619: D605.COM, L605.1
- new net N$620: D606.COM, L606.1
- new net N$621: D607.COM, L607.1
- new net N$622: D608.COM, L608.1
- new net N$623: D609.COM, L609.1
- new net N$624: D610.COM, L610.1
- new net N$625: D611.COM, L611.1
- new net N$626: D612.COM, L612.1
- new net N$627: D613.COM, L613.1
- new net N$628: D614.COM, L614.1
- new net N$629: D615.COM, L615.1
- new net N$630: D616.COM, L616.1
- new net N$631: D617.COM, L617.1
- new net N$632: D618.COM, L618.1
- new net N$633: D619.COM, L619.1
- new net N$634: D620.COM, L620.1
- new net N$635: D621.COM, L621.1
- new net N$636: D622.COM, L622.1
- new net N$637: D623.COM, L623.1
- new net N$638: D624.COM, L624.1
- new net N$639: D625.COM, L625.1
- new net N$640: D626.COM, L626.1
- new net N$641: D627.COM, L627.1
- new net N$642: D628.COM, L628.1
- new net N$643: D629.COM, L629.1
- new net N$644: D630.COM, L630.1
- new net N$645: D631.COM, L631.1
- new net N$646: D632.COM, L632.1
- new net N$647: D633.COM, L633.1
- new net N$648: D634.COM, L634.1
- new net N$649: D635.COM, L635.1
- new net N$650: D636.COM, L636.1
- new net N$651: D637.COM, L637.1
- new net N$652: D638.COM, L638.1
- new net N$653: D639.COM, L639.1
- new net N$654: D640.COM, L640.1
- new net N$655: D641.COM, L641.1
- new net N$656: D642.COM, L642.1
- new net N$657: D643.COM, L643.1
- new net N$658: D644.COM, L644.1
- new net N$659: D645.COM, L645.1
- new net N$660: D646.COM, L646.1
- new net N$661: D647.COM, L647.1
- new net N$662: D648.COM, L648.1
- new net N$663: D649.COM, L649.1
- new net N$664: D650.COM, L650.1
- new net N$665: D651.COM, L651.1
- new net N$666: D652.COM, L652.1
- new net N$667: D653.COM, L653.1
- new net N$668: D654.COM, L654.1
- new net N$669: D655.COM, L655.1
- new net N$670: D656.COM, L656.1
- new net N$671: D657.COM, L657.1
- new net N$672: D658.COM, L658.1
- new net N$673: D659.COM, L659.1
- new net N$674: D660.COM, L660.1
- new net N$675: D661.COM, L661.1
- new net N$676: D662.COM, L662.1
- new net N$677: D663.COM, L663.1
- new net N$678: D664.COM, L664.1
- new net N$679: D665.COM, L665.1
- new net N$680: D666.COM, L666.1
- new net N$681: D667.COM, L667.1
- new net N$682: D668.COM, L668.1
- new net N$683: D669.COM, L669.1
- new net N$684: D670.COM, L670.1
- new net N$685: D671.COM, L671.1
- new net N$686: D672.COM, L672.1
- new net N$687: D673.COM, L673.1
- new net N$688: D674.COM, L674.1
- new net N$689: D675.COM, L675.1
- new net N$690: D676.COM, L676.1
- new net N$691: D677.COM, L677.1
- new net N$692: D678.COM, L678.1
- new net N$693: D679.COM, L679.1
- new net N$694: D680.COM, L680.1
- new net N$695: D681.COM, L681.1
- new net N$696: D682.COM, L682.1
- new net N$697: D683.COM, L683.1
- new net N$698: D684.COM, L684.1
- new net N$699: D685.COM, L685.1
- new net N$700: D686.COM, L686.1
- new net N$701: D687.COM, L687.1
- new net N$702: D688.COM, L688.1
- new net N$703: D689.COM, L689.1
- new net N$704: D690.COM, L690.1
- new net N$705: D691.COM, L691.1
- new net N$706: D692.COM, L692.1
- new net N$707: D693.COM, L693.1
- new net N$708: D694.COM, L694.1
- new net N$709: D695.COM, L695.1
- new net N$710: D696.COM, L696.1
- new net N$711: D697.COM, L697.1
- new net N$712: D698.COM, L698.1
- new net N$713: D699.COM, L699.1
- new net N$714: D700.COM, L700.1
- new net N$715: D701.COM, L701.1
- new net N$716: D702.COM, L702.1
- new net N$717: D703.COM, L703.1
- new net N$718: D704.COM, L704.1
- new net N$719: D705.COM, L705.1
- new net N$720: D706.COM, L706.1
- new net N$721: D707.COM, L707.1
- new net N$722: D708.COM, L708.1
- new net N$723: D709.COM, L709.1
- new net N$724: D710.COM, L710.1
- new net N$725: D711.COM, L711.1
- new net N$726: D712.COM, L712.1
- new net N$727: D713.COM, L713.1
- new net N$728: D714.COM, L714.1
- new net N$729: D715.COM, L715.1
- new net N$730: D716.COM, L716.1
- new net N$731: D717.COM, L717.1
- new net N$732: D718.COM, L718.1
- new net N$733: D719.COM, L719.1
- new net N$734: D720.COM, L720.1
- new net N$735: D721.COM, L721.1
- new net N$736: D722.COM, L722.1
- new net N$737: D723.COM, L723.1
- new net N$738: D724.COM, L724.1
- new net N$739: D725.COM, L725.1
- new net N$740: D726.COM, L726.1
- new net N$741: D727.COM, L727.1
- new net N$742: D728.COM, L728.1
- new net N$743: D729.COM, L729.1
- new net N$744: D730.COM, L730.1
- new net N$745: D731.COM, L731.1
- new net N$746: D732.COM, L732.1
- new net N$747: D733.COM, L733.1
- new net N$748: D734.COM, L734.1
- new net N$749: D735.COM, L735.1
- new net N$750: D736.COM, L736.1
- new net N$751: D737.COM, L737.1
- new net N$752: D738.COM, L738.1
- new net N$753: D739.COM, L739.1
- new net N$754: D740.COM, L740.1
- new net N$755: D741.COM, L741.1
- new net N$756: D742.COM, L742.1
- new net N$757: D743.COM, L743.1
- new net N$758: D744.COM, L744.1
- new net N$759: D745.COM, L745.1
- new net N$760: D746.COM, L746.1
- new net N$761: D747.COM, L747.1
- new net N$762: D748.COM, L748.1
- new net N$763: D749.COM, L749.1
- new net N$764: D750.COM, L750.1
- new net N$765: D751.COM, L751.1
- new net N$766: D752.COM, L752.1
- new net N$767: D753.COM, L753.1
- new net N$768: D754.COM, L754.1
- new net N$769: D755.COM, L755.1
- new net N$770: D756.COM, L756.1
- new net N$771: D757.COM, L757.1
- new net N$772: D758.COM, L758.1
- new net N$773: D759.COM, L759.1
- new net N$774: D760.COM, L760.1
- new net N$775: D761.COM, L761.1
- new net N$776: D762.COM, L762.1
- new net N$777: D763.COM, L763.1
- new net N$778: D764.COM, L764.1
- new net N$779: D765.COM, L765.1
- new net N$780: D766.COM, L766.1
- new net N$781: D767.COM, L767.1
- new net N$782: D768.COM, L768.1
- new net N$783: D769.COM, L769.1
- new net N$784: D770.COM, L770.1
- new net N$785: D771.COM, L771.1
- new net N$786: D772.COM, L772.1
- new net N$787: D773.COM, L773.1
- new net N$788: D774.COM, L774.1
- new net N$789: D775.COM, L775.1
- new net N$79: D65.COM, L65.1
- new net N$790: D776.COM, L776.1
- new net N$791: D777.COM, L777.1
- new net N$792: D778.COM, L778.1
- new net N$793: D779.COM, L779.1
- new net N$794: D780.COM, L780.1
- new net N$795: D781.COM, L781.1
- new net N$796: D782.COM, L782.1
- new net N$797: D783.COM, L783.1
- new net N$798: D784.COM, L784.1
- new net N$799: D785.COM, L785.1
- new net N$80: D66.COM, L66.1
- new net N$800: D786.COM, L786.1
- new net N$801: D787.COM, L787.1
- new net N$802: D788.COM, L788.1
- new net N$803: D789.COM, L789.1
- new net N$804: D790.COM, L790.1
- new net N$805: D791.COM, L791.1
- new net N$806: D792.COM, L792.1
- new net N$807: D793.COM, L793.1
- new net N$808: D794.COM, L794.1
- new net N$809: D795.COM, L795.1
- new net N$81: D67.COM, L67.1
- new net N$810: D796.COM, L796.1
- new net N$811: D797.COM, L797.1
- new net N$812: D798.COM, L798.1
- new net N$813: D799.COM, L799.1
- new net N$814: D800.COM, L800.1
- new net N$815: D801.COM, L801.1
- new net N$816: D802.COM, L802.1
- new net N$817: D803.COM, L803.1
- new net N$818: D804.COM, L804.1
- new net N$819: D805.COM, L805.1
- new net N$82: D68.COM, L68.1
- new net N$820: D806.COM, L806.1
- new net N$821: D807.COM, L807.1
- new net N$822: D808.COM, L808.1
- new net N$823: D809.COM, L809.1
- new net N$824: D810.COM, L810.1
- new net N$825: D811.COM, L811.1
- new net N$826: D812.COM, L812.1
- new net N$827: D813.COM, L813.1
- new net N$828: D814.COM, L814.1
- new net N$829: D815.COM, L815.1
- new net N$83: D69.COM, L69.1
- new net N$830: D816.COM, L816.1
- new net N$831: D817.COM, L817.1
- new net N$832: D818.COM, L818.1
- new net N$833: D819.COM, L819.1
- new net N$834: D820.COM, L820.1
- new net N$835: D821.COM, L821.1
- new net N$836: D822.COM, L822.1
- new net N$837: D823.COM, L823.1
- new net N$838: D824.COM, L824.1
- new net N$839: D825.COM, L825.1
- new net N$84: D70.COM, L70.1
- new net N$840: D826.COM, L826.1
- new net N$841: D827.COM, L827.1
- new net N$842: D828.COM, L828.1
- new net N$843: D829.COM, L829.1
- new net N$844: D830.COM, L830.1
- new net N$845: D831.COM, L831.1
- new net N$846: D832.COM, L832.1
- new net N$847: D833.COM, L833.1
- new net N$848: D834.COM, L834.1
- new net N$849: D835.COM, L835.1
- new net N$85: D71.COM, L71.1
- new net N$850: D836.COM, L836.1
- new net N$851: D837.COM, L837.1
- new net N$852: D838.COM, L838.1
- new net N$853: D839.COM, L839.1
- new net N$854: D840.COM, L840.1
- new net N$855: D841.COM, L841.1
- new net N$856: D842.COM, L842.1
- new net N$857: D843.COM, L843.1
- new net N$858: D844.COM, L844.1
- new net N$859: D845.COM, L845.1
- new net N$86: D72.COM, L72.1
- new net N$860: D846.COM, L846.1
- new net N$861: D847.COM, L847.1
- new net N$862: D848.COM, L848.1
- new net N$863: D849.COM, L849.1
- new net N$864: D850.COM, L850.1
- new net N$865: D851.COM, L851.1
- new net N$866: D852.COM, L852.1
- new net N$867: D853.COM, L853.1
- new net N$868: D854.COM, L854.1
- new net N$869: D855.COM, L855.1
- new net N$87: D73.COM, L73.1
- new net N$870: D856.COM, L856.1
- new net N$871: D857.COM, L857.1
- new net N$872: D858.COM, L858.1
- new net N$873: D859.COM, L859.1
- new net N$874: D860.COM, L860.1
- new net N$875: D861.COM, L861.1
- new net N$876: D862.COM, L862.1
- new net N$877: D863.COM, L863.1
- new net N$878: D864.COM, L864.1
- new net N$879: D865.COM, L865.1
- new net N$88: D74.COM, L74.1
- new net N$880: D866.COM, L866.1
- new net N$881: D867.COM, L867.1
- new net N$882: D868.COM, L868.1
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
Commit message: Wired transistor arrays to correct 18V lines, separated diodes/coils schematic into 4 sheets, add frames
Connections:
- removed net 5V1: IC28.CD+
- removed net 5V2: IC16.CD+, IC19.CD+, IC22.CD+
- removed net 5V3: IC25.CD+
- removed net C13_SOURCE: IC17A.S12
- removed net C16_SOURCE: IC17A.S15
- removed net C17_SINK: IC20A.S0
- removed net C17_SOURCE: IC20A.S8
- removed net C18_SINK: IC20A.S1
- removed net C18_SOURCE: IC20A.S9
- removed net C19_SINK: IC20A.S2
- removed net C19_SOURCE: IC20A.S10
- removed net C1_SINK: IC14A.S0
- removed net C1_SOURCE: IC14A.S8
- removed net C20_SINK: IC20A.S3
- removed net C20_SOURCE: IC20A.S11
- removed net C21_SINK: IC20A.S4
- removed net C21_SOURCE: IC20A.S12
- removed net C22_SINK: IC20A.S5
- removed net C22_SOURCE: IC20A.S13
- removed net C23_SINK: IC20A.S6
- removed net C23_SOURCE: IC20A.S14
- removed net C24_SINK: IC20A.S7
- removed net C24_SOURCE: IC20A.S15
- removed net C25_SINK: IC23A.S0
- removed net C25_SOURCE: IC23A.S8
- removed net C26_SINK: IC23A.S1
- removed net C26_SOURCE: IC23A.S9
- removed net C27_SINK: IC23A.S2
- removed net C27_SOURCE: IC23A.S10
- removed net C28_SINK: IC23A.S3
- removed net C28_SOURCE: IC23A.S11
- removed net C29_SINK: IC23A.S4
- removed net C29_SOURCE: IC23A.S12
- removed net C2_SINK: IC14A.S1
- removed net C2_SOURCE: IC14A.S9
- removed net C30_SINK: IC23A.S5
- removed net C30_SOURCE: IC23A.S13
- removed net C31_SINK: IC23A.S6
- removed net C31_SOURCE: IC23A.S14
- removed net C32_SINK: IC23A.S7
- removed net C32_SOURCE: IC23A.S15
- removed net C3_SINK: IC14A.S2
- removed net C3_SOURCE: IC14A.S10
- removed net C4_SINK: IC14A.S3
- removed net C4_SOURCE: IC14A.S11
- removed net C5_SINK: IC14A.S4
- removed net C5_SOURCE: IC14A.S12
- removed net C6_SINK: IC14A.S5
- removed net C6_SOURCE: IC14A.S13
- removed net C7_SINK: IC14A.S6
- removed net C7_SOURCE: IC14A.S14
- removed net C8_SINK: IC14A.S7
- removed net C8_SOURCE: IC14A.S15
- removed net COL25_SINK: IC24.O1
- removed net COL25_SOURCE: IC25.O1
- removed net COL26_SINK: IC24.O2
- removed net COL26_SOURCE: IC25.O2
- removed net COL27_SINK: IC24.O3
- removed net COL27_SOURCE: IC25.O3
- removed net COL28_SINK: IC24.O4
- removed net COL28_SOURCE: IC25.O4
- removed net COL29_SINK: IC24.O5
- removed net COL29_SOURCE: IC25.O5
- removed net COL30_SINK: IC24.O6
- removed net COL30_SOURCE: IC25.O6
- removed net COL31_SINK: IC24.O7
- removed net COL31_SOURCE: IC25.O7
- removed net COL32_SINK: IC24.O8
- removed net COL32_SOURCE: IC25.O8
- removed net N$16: IC24.I5
- removed net N$4: IC27.I5
- removed net R1_SINK3: IC28.I1
- removed net R1_SINK5: IC19.I1
- removed net R1_SINK7: IC25.I1
- removed net R1_SOURCE3: IC27.I1
- removed net R1_SOURCE5: IC18.I1
- removed net R1_SOURCE7: IC24.I1
- removed net R2_SINK3: IC28.I2
- removed net R2_SINK5: IC19.I2
- removed net R2_SINK7: IC25.I2
- removed net R2_SOURCE3: IC27.I2
- removed net R2_SOURCE5: IC18.I2
- removed net R2_SOURCE7: IC24.I2
- removed net R3_SINK3: IC28.I3
- removed net R3_SINK5: IC19.I3
- removed net R3_SINK7: IC25.I3
- removed net R3_SOURCE3: IC27.I3
- removed net R3_SOURCE5: IC18.I3
- removed net R3_SOURCE7: IC24.I3
- removed net R4_SINK3: IC28.I4
- removed net R4_SINK5: IC19.I4
- removed net R4_SINK7: IC25.I4
- removed net R4_SOURCE3: IC27.I4
- removed net R4_SOURCE5: IC18.I4
- removed net R4_SOURCE7: IC24.I4
- removed net R5_SINK3: IC28.I5
- removed net R5_SINK5: IC19.I5
- removed net R5_SINK7: IC25.I5
- removed net R6_SINK3: IC28.I6
- removed net R6_SINK5: IC19.I6
- removed net R6_SINK7: IC25.I6
- removed net R6_SOURCE3: IC27.I6
- removed net R6_SOURCE5: IC18.I6
- removed net R6_SOURCE7: IC24.I6
- removed net R7_SINK3: IC28.I7
- removed net R7_SINK5: IC19.I7
- removed net R7_SINK7: IC25.I7
- removed net R7_SOURCE3: IC27.I7
- removed net R7_SOURCE5: IC18.I7
- removed net R7_SOURCE7: IC24.I7
- removed net R8_SINK3: IC28.I8
- removed net R8_SINK5: IC19.I8
- removed net R8_SINK7: IC25.I8
- removed net R8_SOURCE3: IC27.I8
- removed net R8_SOURCE7: IC24.I8
- removed net VCC: IC10.VCC, IC12.VCC, IC15.VCC, IC18.VCC, IC21.VCC, IC24.VCC, IC27.VCC, IC7.VCC
- new net R25_SINK1: IC23A.S0, IC25.I1
- new net R25_SOURCE1: IC23A.S8, IC24.I1
- new net R26_SINK1: IC23A.S1, IC25.I2
- new net R26_SOURCE1: IC23A.S9, IC24.I2
- new net R27_SINK1: IC23A.S2, IC25.I3
- new net R27_SOURCE1: IC23A.S10, IC24.I3
- new net R28_SINK1: IC23A.S3, IC25.I4
- new net R28_SOURCE1: IC23A.S11, IC24.I4
- new net R29_SINK1: IC23A.S4, IC25.I5
- new net R29_SOURCE1: IC23A.S12, IC24.I5
- new net R30_SINK1: IC23A.S5, IC25.I6
- new net R30_SOURCE1: IC23A.S13, IC24.I6
- new net R31_SINK1: IC23A.S6, IC25.I7
- new net R31_SOURCE1: IC23A.S14, IC24.I7
- new net R32_SINK1: IC23A.S7, IC25.I8
- new net R32_SOURCE1: IC23A.S15, IC24.I8
- net 18V_PULSE_1: now also IC10.VCC, IC12.VCC, IC13.CD+, IC15.VCC, IC18.VCC, IC21.VCC, IC24.VCC, IC27.VCC, IC28.CD+, IC6.CD+, IC7.VCC, IC9.CD+
- net 18V_PULSE_2: now also IC16.CD+, IC19.CD+, IC22.CD+, IC25.CD+
- net 5V: no longer IC13.CD+, IC6.CD+, IC9.CD+
- net C10_SINK: now also IC19.I2
- net C10_SOURCE: now also IC18.I2
- net C11_SINK: now also IC19.I3
- net C11_SOURCE: now also IC18.I3
- net C12_SINK: now also IC19.I4
- net C12_SOURCE: now also IC18.I4
- net C13_SINK: now also IC19.I5
- net C14_SINK: now also IC19.I6
- net C14_SOURCE: now also IC18.I6
- net C15_SINK: now also IC19.I7
- net C15_SOURCE: now also IC18.I7
- net C16_SINK: now also IC19.I8
- net C9_SINK: now also IC19.I1
- net C9_SOURCE: now also IC18.I1
- net COL25: now also IC24.O1, IC25.O1
- net COL26: now also IC24.O2, IC25.O2
- net COL27: now also IC24.O3, IC25.O3
- net COL28: now also IC24.O4, IC25.O4
- net COL29: now also IC24.O5, IC25.O5
- net COL30: now also IC24.O6, IC25.O6
- net COL31: now also IC24.O7, IC25.O7
- net COL32: now also IC24.O8, IC25.O8
- net N$11: now also IC14A.S12
- net N$13: now also IC17A.S12
- net N$14: now also IC20A.S12
- net R1_SINK4: now also IC14A.S0
- net R1_SINK6: now also IC20A.S0
- net R1_SOURCE4: now also IC14A.S8
- net R1_SOURCE6: now also IC20A.S8
- net R25_SINK: now also IC28.I1
- net R25_SOURCE: now also IC27.I1
- net R26_SINK: now also IC28.I2
- net R26_SOURCE: now also IC27.I2
- net R27_SINK: now also IC28.I3
- net R27_SOURCE: now also IC27.I3
- net R28_SINK: now also IC28.I4
- net R28_SOURCE: now also IC27.I4
- net R29_SINK: now also IC28.I5
- net R29_SOURCE: now also IC27.I5
- net R2_SINK4: now also IC14A.S1
- net R2_SINK6: now also IC20A.S1
- net R2_SOURCE4: now also IC14A.S9
- net R2_SOURCE6: now also IC20A.S9
- net R30_SINK: now also IC28.I6
- net R30_SOURCE: now also IC27.I6
- net R31_SINK: now also IC28.I7
- net R31_SOURCE: now also IC27.I7
- net R32_SINK: now also IC28.I8
- net R32_SOURCE: now also IC27.I8
- net R3_SINK4: now also IC14A.S2
- net R3_SINK6: now also IC20A.S2
- net R3_SOURCE4: now also IC14A.S10
- net R3_SOURCE6: now also IC20A.S10
- net R4_SINK4: now also IC14A.S3
- net R4_SINK6: now also IC20A.S3
- net R4_SOURCE4: now also IC14A.S11
- net R4_SOURCE6: now also IC20A.S11
- net R5_SINK4: now also IC14A.S4
- net R5_SINK6: now also IC20A.S4
- net R6_SINK4: now also IC14A.S5
- net R6_SINK6: now also IC20A.S5
- net R6_SOURCE4: now also IC14A.S13
- net R6_SOURCE6: now also IC20A.S13
- net R7_SINK4: now also IC14A.S6
- net R7_SINK6: now also IC20A.S6
- net R7_SOURCE4: now also IC14A.S14
- net R7_SOURCE6: now also IC20A.S14
- net R8_SINK4: now also IC14A.S7
- net R8_SINK6: now also IC20A.S7
- net R8_SOURCE4: now also IC14A.S15
- net R8_SOURCE5: now also IC17A.S15
- net R8_SOURCE6: now also IC20A.S15
